File: Schematics/Audio _Eagle/Amplifier_v1.1.brd (EAGLE design)
At the start: 100 x 80 mm, 100 parts, among them U1 NE5532, U2 NE5532, U3 NE5532, U4 NE5532, U5 NE5532, U6 NE5532, U7 NE5532, U8 LME49830

Commit message: update to amp schematic
Parts:
- removed R39: (no value), resistor:0207/7
- removed R40, R41, R42: (no value), pot:3RP/1610G
- removed U1, U2, U3, U4, U5, U6, U7: NE5532, NE5532:DIL08
- added C22, C23, C27: 100uF, rcl:E2,5-6
- added C24, C25, C26: 0.1uF, rcl:C025-024X044
- added C29, C31, C33, C35, C37, C39, C41, C43, C45, C47, C49, C51, C53, C55: 10uF, rcl:C025-024X044
- added IC1, IC2, IC3, IC4, IC5, IC6, IC7: NE5532N, linear:DIL08
- added R51: 10, rcl:0204V
- added R52: 1.2k, rcl:0204V
- added U$13, U$14: TONE_POT_2GANG, Amplifier_Parts:TONE_POT_2GANG
- added U$15: INDUCTOR, Amplifier_Parts:INDUCTOR
- added U$16: VOL_POT_2GANG, Amplifier_Parts:VOL_POT_2GANG
- R1, R10, R11, R12, R13, R14, R15, R16, R17, R18, R19, R2, R20, R21, R22, R23, R24, R25, R26, R27, R28, R29, R30, R31, R32, R33, R34, R35, R36, R37, R38, R4, R44, R45, R47, R48, R49, R5, R50, R6, R7, R8, R9: device resistor:0207/7 -> rcl:0204V
- R3: device pot:3RP/1610G -> rcl:0204V
- R46: value 1.2k -> 12k; device resistor:0207/7 -> rcl:0204V
- U$1: value INDUCTOR -> TONE_POT_2GANG; device Amplifier_Parts:INDUCTOR -> Amplifier_Parts:TONE_POT_2GANG
- moved C10 498.2 mm to (-106.7, -402.6)
- moved C11 497.5 mm to (-101.6, -402.6)
- moved C12 497.0 mm to (-96.5, -402.6)
- moved C13 496.7 mm to (-91.4, -402.6)
- moved C15 496.7 mm to (-81.3, -402.6)
- moved C14 496.6 mm to (-86.4, -402.6)
- moved R32 492.3 mm to (-104.1, -397.5)
- moved R33 489.6 mm to (-94.0, -397.5)
- moved R38 487.1 mm to (-63.5, -397.5)
- moved R36 486.6 mm to (-83.8, -397.5)
- moved R37 486.4 mm to (-73.7, -397.5)
- moved R31 483.5 mm to (-63.5, -392.4)
- moved R27 478.4 mm to (-104.1, -392.4)
- moved R23 477.3 mm to (-94.0, -387.4)
- moved R28 476.9 mm to (-94.0, -392.4)
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Connections:
- removed net +VCC: U8.15
- removed net -VEE: U8.10
- removed net N$10: R6.1, R8.2, U2.1
- removed net N$16: C7.2, C8.2, U$5.1
- removed net N$20: R10.1, U$3.1, U$4.1
- removed net N$26: R16.2, R36.1, U4.8
- removed net N$28: R15.1, U$6.1
- removed net N$31: C10.1, C11.1, R20.1
- removed net N$36: C12.2, R24.2, U$8.2
- removed net N$39: R26.1, R27.2, U6.1
- removed net N$4: C10.2, R19.2, U$1.1
- removed net N$40: R26.2, R38.1, U6.8
- removed net N$48: U7.5
- removed net N$51: C13.1, U$12.1
- removed net N$52: C9.2, R19.1, R24.1, R29.1
- removed net N$62: R38.2, R41.2-1
- removed net N$63 (its old number): R42.2-2, R42.2-3, U7.7
- removed net N$8: C3.1, C4.1, R5.1
- new net N$30: IC4.6, R19.2, R29.1
- new net N$80: C17.2, C2.-, U8.10
- new net N$82: C16.+, C18.1, U8.15
- new net N$84: C26.2, R51.1
- new net N$85: C27.+, R52.2, U8.2
- new net N$88: IC1.1, R6.1, R8.2
- new net VCC: C22.+, C24.1, C31.1, C35.1, C39.1, C43.1, C47.1, C51.1, C55.1, IC1.8, IC2.8, IC3.8, IC4.8, IC5.8, IC6.8, IC7.8, P_D.PAD
- new net VEE: C23.-, C25.2, C29.2, C33.2, C37.2, C41.2, C45.2, C49.2, C53.2, IC1.4, IC2.4, IC3.4, IC4.4, IC5.4, IC6.4, IC7.4, N_D.PAD
- net GND: now also C10.1, C11.1, C14.2, C15.2, C16.-, C17.1, C18.2, C2.+, C22.-, C23.+, C24.2, C25.1, C26.1, C27.-, C29.1, C3.1, C31.2, C33.1, C35.2, C37.1, C39.2, C4.1, C41.1, C43.2, C45.1, C47.2, C49.1, C51.2, C53.1, C55.2, C7.2, C8.2, IC1.5, IC2.5, IC3.5, IC4.5, IC5.5, IC6.5, IC7.3, IC7.5, R10.1, R13.1, R15.1, R20.1, R23.1, R26.1, R28.1, R3.2, R31.2, R38.1, R5.1, R7.1, U$10.1, U$11.1, U$12.1, U$3.1, U$4.1, U$5.1, U$6.1, U$9.1
- net N$1: now also IC7.2, U$16.1_1; no longer R3.2-1, U1.2
- net N$11: now also IC1.6; no longer U2.8
- net N$12: now also C3.2, IC1.3, R3.1, U$2.1; no longer U2.5
- net N$14: now also IC2.3; no longer U3.3
- net N$15: now also IC3.1, R16.1, R17.2; no longer R12.1, R13.2, U3.2
- net N$17: now also IC2.1; no longer U3.1
- net N$18: now also IC2.6; no longer U3.8
- net N$19: now also IC3.6, R16.2, R18.1; no longer U3.5
- net N$2: now also IC7.1, U$16.1_2, U$16.1_3; no longer R3.2-2, R3.2-3, U1.1
- net N$21: now also IC3.7, U$14.1_2, U$14.1_3; no longer C11.2, R20.2, U$1.2, U5.3
- net N$23: now also IC3.3; no longer U4.3
- net N$24: now also U$14.1_1; no longer R17.1, U4.2
- net N$25: now also C11.2, R32.2, U$8.2; no longer R16.1, R17.2, U4.1
- net N$27: now also IC3.2, R17.1, R5.2; no longer U4.5
- net N$3: now also IC7.6, U$16.2_1; no longer R3.1-1, U1.8
- net N$32: now also C12.2, U$9.2; no longer R23.1, U5.2
- net N$33: now also C12.1, IC5.3, U$10.2; no longer R21.1, U5.1
- net N$34: now also IC5.1, R24.1, R25.2; no longer R21.2, R37.1, U5.8
- net N$35: now also IC5.6, R24.2, R30.1; no longer U5.5
- net N$37: now also C13.2, C15.1, R27.2, U$11.2; no longer C12.1, R25.2, U$9.2, U6.3
- net N$38: now also C14.1, IC6.3, U$12.2, U$15.2; no longer R27.1, U6.2
- net N$41: now also C13.1, U$15.1; no longer U6.5
- net N$42: now also R29.2, U$1.2_1; no longer R25.1, U$8.1, U$9.1
- net N$43: now also IC4.7, U$1.2_2, U$1.2_3; no longer C13.2, C15.1, R29.2, U$10.2
- net N$44: now also IC5.7, U$13.2_2, U$13.2_3; no longer C14.1, R30.2, U$11.2, U$12.2, U7.3
- net N$45: now also R30.2, U$13.2_1; no longer R32.1, R33.2, U7.2
- net N$46: now also IC4.1, R19.1, R21.2; no longer R31.1, R32.2, U7.1
- net N$47: now also C10.2, IC4.3, R31.1, U$8.1; no longer R31.2, R39.1, U7.8
- net N$49: now also IC4.2, R20.2, R21.1; no longer R30.1, U$11.1
- net N$5: now also IC7.7, U$16.2_2, U$16.2_3; no longer R3.1-2, R3.1-3, U1.7
- net N$50: now also IC5.2, R25.1, R26.2; no longer C14.2, C15.2, U$10.1
- net N$53: now also U$1.1_1; no longer R40.1-1
- net N$54: now also IC1.7, U$1.1_2, U$1.1_3; no longer R40.1-2, R40.1-3, U2.7
- net N$55: now also IC2.7, U$13.1_2, U$13.1_3; no longer R41.1-2, R41.1-3, U3.7
- net N$56: now also U$13.1_1; no longer R41.1-1
- net N$57: now also IC6.1, R33.1, R36.2; no longer R42.1-2, R42.1-3, U4.7
- net N$58: now also IC6.6, R33.2, R37.1; no longer R36.2, R42.1-1
- net N$59: now also IC6.7, U$14.2_2, U$14.2_3; no longer R40.2-2, R40.2-3, U5.7
- net N$6: now also IC1.2, R7.2, R8.1; no longer C3.2, R4.2, U$2.1
- net N$60: now also U$14.2_1; no longer R40.2-1
- net N$61: now also IC6.2, R36.1, R38.2; no longer R41.2-2, R41.2-3, U6.7
- net N$64: now also C9.2, R22.1, R27.1, R32.1; no longer R39.2, R42.2-1
- net N$7: now also R4.2; no longer R5.2, U2.3
- net N$74: now also P_S.PAD; no longer P_D.PAD
- net N$75: now also N_S.PAD, R51.2; no longer N_D.PAD
- net N$9: now also IC2.2, R12.1, R13.2; no longer R7.2, R8.1, U2.2

Commit message: updated schematic
Parts:
- added IC8: LM317MABDTRK, v-reg:DPACK
- added IC9: LM337, Amplifier_Parts:LM337
- C29, C31, C33, C35, C37, C39, C41, C43, C45, C47, C49, C51, C53, C55: value 10uF -> 0.1uF
Changed lines of the file:
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@@
 <element name="U$13" library="Amplifier_Parts" package="TONE_POT_2GANG" value="TONE_POT_2GANG" x="-99.06" y="-416.56"/>
 <element name="U$14" library="Amplifier_Parts" package="TONE_POT_2GANG" value="TONE_POT_2GANG" x="-99.06" y="-425.45"/>
-<element name="C29" library="rcl" package="C025-024X044" value="10uF" x="-106.68" y="-440.69"/>
-<element name="C31" library="rcl" package="C025-024X044" value="10uF" x="-106.68" y="-454.66"/>
-<element name="C33" library="rcl" package="C025-024X044" value="10uF" x="-106.68" y="-476.25"/>
-<element name="C35" library="rcl" package="C025-024X044" value="10uF" x="-100.33" y="-476.25"/>
-<element name="C37" library="rcl" package="C025-024X044" value="10uF" x="-106.68" y="-497.84"/>
-<element name="C39" library="rcl" package="C025-024X044" value="10uF" x="-100.33" y="-497.84"/>
-<element name="C41" library="rcl" package="C025-024X044" value="10uF" x="-106.68" y="-519.43"/>
-<element name="C43" library="rcl" package="C025-024X044" value="10uF" x="-100.33" y="-519.43"/>
-<element name="C45" library="rcl" package="C025-024X044" value="10uF" x="-106.68" y="-541.02"/>
-<element name="C47" library="rcl" package="C025-024X044" value="10uF" x="-100.33" y="-541.02"/>
-<element name="C49" library="rcl" package="C025-024X044" value="10uF" x="-106.68" y="-562.61"/>
-<element name="C51" library="rcl" package="C025-024X044" value="10uF" x="-100.33" y="-562.61"/>
-<element name="C53" library="rcl" package="C025-024X044" value="10uF" x="-106.68" y="-584.2"/>
-<element name="C55" library="rcl" package="C025-024X044" value="10uF" x="-100.33" y="-584.2"/>
+<element name="C29" library="rcl" package="C025-024X044" value="0.1uF" x="-106.68" y="-440.69"/>
+<element name="C31" library="rcl" package="C025-024X044" value="0.1uF" x="-106.68" y="-454.66"/>
+<element name="C33" library="rcl" package="C025-024X044" value="0.1uF" x="-106.68" y="-476.25"/>
+<element name="C35" library="rcl" package="C025-024X044" value="0.1uF" x="-100.33" y="-476.25"/>
+<element name="C37" library="rcl" package="C025-024X044" value="0.1uF" x="-106.68" y="-497.84"/>
+<element name="C39" library="rcl" package="C025-024X044" value="0.1uF" x="-100.33" y="-497.84"/>
+<element name="C41" library="rcl" package="C025-024X044" value="0.1uF" x="-106.68" y="-519.43"/>
+<element name="C43" library="rcl" package="C025-024X044" value="0.1uF" x="-100.33" y="-519.43"/>
+<element name="C45" library="rcl" package="C025-024X044" value="0.1uF" x="-106.68" y="-541.02"/>
+<element name="C47" library="rcl" package="C025-024X044" value="0.1uF" x="-100.33" y="-541.02"/>
+<element name="C49" library="rcl" package="C025-024X044" value="0.1uF" x="-106.68" y="-562.61"/>
+<element name="C51" library="rcl" package="C025-024X044" value="0.1uF" x="-100.33" y="-562.61"/>
+<element name="C53" library="rcl" package="C025-024X044" value="0.1uF" x="-106.68" y="-584.2"/>
+<element name="C55" library="rcl" package="C025-024X044" value="0.1uF" x="-100.33" y="-584.2"/>
+<element name="IC8" library="v-reg" package="DPACK" value="LM317MABDTRK" x="-115.57" y="-580.39"/>
+<element name="IC9" library="Amplifier_Parts" package="LM337" value="LM337" x="-127" y="-580.39"/>
 </elements>
 <signals>

Commit message: amp schematic updates
Parts:
- added C28, C30, C32, C34, C36, C38: 100uF, rcl:E2,5-6
- added C40, C42: 0.1uF, rcl:C025-024X044
- added R39, R40, R41, R42: (no value), rcl:0204V
- added R53, R54, R55, R56: 1.2k, rcl:0204V
- added R57: (no value), pot:B25U
- added U$17: MOLEX_6P, Amplifier_Parts:MOLEX_6P
Connections:
- net N$82 renamed V+
- removed net N$71: R48.2, U8.8
- removed net N$80: C17.2, C2.-, U8.10
- removed net VEE: C23.-, C25.2, C29.2, C33.2, C37.2, C41.2, C45.2, C49.2, C53.2, IC1.4, IC2.4, IC3.4, IC4.4, IC5.4, IC6.4, IC7.4, N_D.PAD
- new net +12V: C31.1, C32.+, C35.1, C36.+, C39.1, C43.1, C47.1, C51.1, C55.1, IC1.8, IC2.8, IC3.8, IC4.8, IC5.8, IC6.8, IC7.8, IC8.3
- new net -12V: C29.2, C33.2, C34.-, C37.2, C38.-, C41.2, C45.2, C49.2, C53.2, IC1.4, IC2.4, IC3.4, IC4.4, IC5.4, IC6.4, IC7.4, IC9.4
- new net N$10: IC8.1, R39.1, R40.2
- new net N$16: C40.2, R53.1, R54.1, U8.4
- new net N$20: C28.+, IC8.4, R39.2
- new net N$26: IC9.1, R41.1, R42.2
- new net N$28: C30.-, IC9.3, R41.2
- new net N$31: R55.1, R57.A, U8.5
- new net N$36: C42.2, R55.2
- new net N$4: R48.2, U8.14
- new net N$40: R56.2, R57.E, R57.S
- new net N$8: C22.-, C24.2
- new net V-: C17.2, C2.-, C23.-, C25.2, N_D.PAD, U8.10
- net GND: now also C28.-, C30.+, C32.-, C34.+, C36.-, C38.+, C40.1, C42.1, R40.1, R42.1, R53.2, U$17.P$2; no longer C22.-, C24.2
- net N$68: now also R43.S
- net N$75: now also R56.1, U$17.P$1, U8.8
- net VCC: no longer C31.1, C35.1, C39.1, C43.1, C47.1, C51.1, C55.1, IC1.8, IC2.8, IC3.8, IC4.8, IC5.8, IC6.8, IC7.8

Commit message: updated schematic
Connections:
- removed net N$20: C28.+, IC8.4, R39.2
- removed net N$28: C30.-, IC9.3, R41.2
- removed net N$8: C22.-, C24.2
- net +12V: now also C28.+, IC8.4, R39.2; no longer C32.+, IC8.3
- net -12V: now also C30.-, IC9.3, R41.2; no longer C34.-, IC9.4
- net GND: now also C22.-, C24.2
- net V+: now also C32.+, IC8.3
- net V-: now also C34.-, IC9.4
Changed lines of the file:
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@@
 <?xml version="1.0" encoding="utf-8"?>
 <!DOCTYPE eagle SYSTEM "eagle.dtd">
-<eagle version="6.5.0">
+<eagle version="7.1.0">
 <drawing>
 <settings>
@@
 <layer number="54" name="bGND_GNDA" color="1" fill="9" visible="no" active="no"/>
 <layer number="56" name="wert" color="7" fill="1" visible="no" active="no"/>
-<layer number="90" name="Modules" color="5" fill="1" visible="yes" active="yes"/>
+<layer number="90" name="Modules" color="5" fill="1" visible="no" active="no"/>
 <layer number="91" name="Nets" color="2" fill="1" visible="no" active="no"/>
 <layer number="92" name="Busses" color="1" fill="1" visible="no" active="no"/>
@@
 <pass name="Default">
 <param name="RoutingGrid" value="50mil"/>
+<param name="AutoGrid" value="1"/>
+<param name="Efforts" value="0"/>
+<param name="TopRouterVariant" value="1"/>
 <param name="tpViaShape" value="round"/>
 <param name="PrefDir.1" value="|"/>
@@
 <contactref element="C16" pad="-"/>
 <contactref element="U$17" pad="P$2"/>
-<wire x1="-102.87" y1="-161.29" x2="-101.6" y2="-148.59" width="0" layer="19" extent="1-1"/>
+<contactref element="C22" pad="-"/>
+<contactref element="C24" pad="2"/>
+<wire x1="-100.33" y1="-154.94" x2="-101.6" y2="-148.59" width="0" layer="19" extent="1-1"/>
+<wire x1="-102.87" y1="-161.29" x2="-100.33" y2="-154.94" width="0" layer="19" extent="1-1"/>
+<wire x1="-99.06" y1="-140.97" x2="-101.6" y2="-148.59" width="0" layer="19" extent="1-1"/>
 <wire x1="-102.87" y1="-172.72" x2="-102.87" y2="-161.29" width="0" layer="19" extent="1-1"/>
 <wire x1="-99.06" y1="-180.34" x2="-102.87" y2="-172.72" width="0" layer="19" extent="1-1"/>
@@
 <wire x1="-130.81" y1="-679.45" x2="-128.27" y2="-660.4" width="0" layer="19" extent="1-1"/>
 <wire x1="-152.01" y1="-677.03" x2="-130.81" y2="-679.45" width="0" layer="19" extent="1-1"/>
-<wire x1="-91.44" y1="-27.94" x2="-101.6" y2="-148.59" width="0" layer="19" extent="1-1"/>
+<wire x1="-91.44" y1="-27.94" x2="-99.06" y2="-140.97" width="0" layer="19" extent="1-1"/>
 <wire x1="-93.98" y1="-22.86" x2="-91.44" y2="-27.94" width="0" layer="19" extent="1-1"/>
 <wire x1="-90.17" y1="-16.51" x2="-93.98" y2="-22.86" width="0" layer="19" extent="1-1"/>
@@
 <contactref element="C17" pad="2"/>
 <contactref element="C2" pad="-"/>
-<wire x1="-100.33" y1="-161.29" x2="-99.06" y2="-148.59" width="0" layer="19" extent="1-1"/>
+<contactref element="IC9" pad="4"/>
+<contactref element="C34" pad="-"/>
+<wire x1="-127" y1="-578.01" x2="-128.27" y2="-632.46" width="0" layer="19" extent="1-1"/>
+<wire x1="-100.33" y1="-161.29" x2="-127" y2="-578.01" width="0" layer="19" extent="1-1"/>
+<wire x1="-99.06" y1="-148.59" x2="-100.33" y2="-161.29" width="0" layer="19" extent="1-1"/>
 <wire x1="-100.33" y1="-124.46" x2="-99.06" y2="-148.59" width="0" layer="19" extent="1-1"/>
 <wire x1="-91.44" y1="-22.86" x2="-100.33" y2="-124.46" width="0" layer="19" extent="1-1"/>
@@
 <wire x1="-117.85" y1="-585.19" x2="-130.81" y2="-590.55" width="0" layer="19" extent="1-1"/>
 </signal>
-<signal name="N$20">
-<contactref element="IC8" pad="4"/>
-<contactref element="R39" pad="2"/>
-<contactref element="C28" pad="+"/>
-<wire x1="-128.27" y1="-590.55" x2="-130.81" y2="-600.71" width="0" layer="19" extent="1-1"/>
-<wire x1="-115.57" y1="-578.01" x2="-128.27" y2="-590.55" width="0" layer="19" extent="1-1"/>
-</signal>
 <signal name="N$26">
 <contactref element="R41" pad="1"/>
@@
 <wire x1="-129.28" y1="-585.19" x2="-130.81" y2="-622.3" width="0" layer="19" extent="1-1"/>
 </signal>
-<signal name="N$28">
-<contactref element="R41" pad="2"/>
-<contactref element="C30" pad="-"/>
-<contactref element="IC9" pad="3"/>
-<wire x1="-128.27" y1="-608.33" x2="-128.27" y2="-622.3" width="0" layer="19" extent="1-1"/>
-<wire x1="-124.72" y1="-585.19" x2="-128.27" y2="-608.33" width="0" layer="19" extent="1-1"/>
-</signal>
 <signal name="-12V">
-<contactref element="IC9" pad="4"/>
-<contactref element="C34" pad="-"/>
 <contactref element="C53" pad="2"/>
 <contactref element="C49" pad="2"/>
@@
 <contactref element="IC7" pad="4"/>
 <contactref element="C38" pad="-"/>
-<wire x1="-128.27" y1="-647.7" x2="-128.27" y2="-632.46" width="0" layer="19" extent="1-1"/>
-<wire x1="-105.41" y1="-584.2" x2="-128.27" y2="-632.46" width="0" layer="19" extent="1-1"/>
+<contactref element="IC9" pad="3"/>
+<contactref element="C30" pad="-"/>
+<contactref element="R41" pad="2"/>
+<wire x1="-128.27" y1="-608.33" x2="-128.27" y2="-622.3" width="0" layer="19" extent="1-1"/>
+<wire x1="-124.72" y1="-585.19" x2="-128.27" y2="-608.33" width="0" layer="19" extent="1-1"/>
+<wire x1="-105.41" y1="-584.2" x2="-124.72" y2="-585.19" width="0" layer="19" extent="1-1"/>
 <wire x1="-105.41" y1="-562.61" x2="-105.41" y2="-584.2" width="0" layer="19" extent="1-1"/>
 <wire x1="-105.41" y1="-541.02" x2="-105.41" y2="-562.61" width="0" layer="19" extent="1-1"/>
@@
 <wire x1="-105.41" y1="-497.84" x2="-105.41" y2="-519.43" width="0" layer="19" extent="1-1"/>
 <wire x1="-105.41" y1="-476.25" x2="-105.41" y2="-497.84" width="0" layer="19" extent="1-1"/>
-<wire x1="-127" y1="-578.01" x2="-105.41" y2="-584.2" width="0" layer="19" extent="1-1"/>
+<wire x1="-128.27" y1="-647.7" x2="-128.27" y2="-622.3" width="0" layer="19" extent="1-1"/>
 <wire x1="-105.41" y1="-440.69" x2="-105.41" y2="-476.25" width="0" layer="19" extent="1-1"/>
 <wire x1="-97.79" y1="-364.49" x2="-105.41" y2="-440.69" width="0" layer="19" extent="1-1"/>
@@
 </signal>
 <signal name="+12V">
-<contactref element="C32" pad="+"/>
-<contactref element="IC8" pad="3"/>
 <contactref element="C31" pad="1"/>
 <contactref element="IC1" pad="8"/>
@@
 <contactref element="IC7" pad="8"/>
 <contactref element="C36" pad="+"/>
-<wire x1="-130.81" y1="-640.08" x2="-130.81" y2="-615.95" width="0" layer="19" extent="1-1"/>
-<wire x1="-113.29" y1="-585.19" x2="-130.81" y2="-615.95" width="0" layer="19" extent="1-1"/>
-<wire x1="-101.6" y1="-584.2" x2="-113.29" y2="-585.19" width="0" layer="19" extent="1-1"/>
-<wire x1="-101.6" y1="-562.61" x2="-101.6" y2="-584.2" width="0" layer="19" extent="1-1"/>
+<contactref element="IC8" pad="4"/>
+<contactref element="R39" pad="2"/>
+<contactref element="C28" pad="+"/>
+<wire x1="-128.27" y1="-590.55" x2="-130.81" y2="-600.71" width="0" layer="19" extent="1-1"/>
+<wire x1="-115.57" y1="-578.01" x2="-128.27" y2="-590.55" width="0" layer="19" extent="1-1"/>
+<wire x1="-101.6" y1="-584.2" x2="-115.57" y2="-578.01" width="0" layer="19" extent="1-1"/>
+<wire x1="-101.6" y1="-562.61" x2="-115.57" y2="-578.01" width="0" layer="19" extent="1-1"/>
 <wire x1="-101.6" y1="-541.02" x2="-101.6" y2="-562.61" width="0" layer="19" extent="1-1"/>
 <wire x1="-101.6" y1="-519.43" x2="-101.6" y2="-541.02" width="0" layer="19" extent="1-1"/>
@@
 <wire x1="-101.6" y1="-476.25" x2="-101.6" y2="-497.84" width="0" layer="19" extent="1-1"/>
 <wire x1="-107.95" y1="-454.66" x2="-101.6" y2="-476.25" width="0" layer="19" extent="1-1"/>
+<wire x1="-130.81" y1="-640.08" x2="-130.81" y2="-600.71" width="0" layer="19" extent="1-1"/>
 <wire x1="-105.41" y1="-356.87" x2="-107.95" y2="-454.66" width="0" layer="19" extent="1-1"/>
 <wire x1="-92.71" y1="-356.87" x2="-105.41" y2="-356.87" width="0" layer="19" extent="1-1"/>
@@
 <wire x1="-105.41" y1="-228.6" x2="-105.41" y2="-279.4" width="0" layer="19" extent="1-1"/>
 <wire x1="-105.41" y1="-218.44" x2="-105.41" y2="-228.6" width="0" layer="19" extent="1-1"/>
-</signal>
-<signal name="N$8">
-<contactref element="C22" pad="-"/>
-<contactref element="C24" pad="2"/>
-<wire x1="-100.33" y1="-154.94" x2="-99.06" y2="-140.97" width="0" layer="19" extent="1-1"/>
 </signal>
 <signal name="N$4">
@@
 <contactref element="C18" pad="1"/>
 <contactref element="U8" pad="15"/>
+<contactref element="C32" pad="+"/>
+<contactref element="IC8" pad="3"/>
+<wire x1="-113.29" y1="-585.19" x2="-130.81" y2="-615.95" width="0" layer="19" extent="1-1"/>
+<wire x1="-93.98" y1="-27.94" x2="-113.29" y2="-585.19" width="0" layer="19" extent="1-1"/>
 <wire x1="-92.71" y1="-16.51" x2="-93.98" y2="-27.94" width="0" layer="19" extent="1-1"/>
 <wire x1="-76.61" y1="-5.08" x2="-92.71" y2="-16.51" width="0" layer="19" extent="1-1"/>
