File: Schematics/Audio _Eagle/Amplifier_v1.1.brd (EAGLE design)
At the start: 100 x 80 mm, 236 parts, among them IC1 NE5532N, IC10 NE5532N, IC11 NE5532N, IC12 NE5532N, IC13 NE5532N, IC2 NE5532N, IC3 NE5532N, IC4 NE5532N, IC5 NE5532N, IC6 NE5532N, IC7 NE5532N, IC8 LM317MABDTRK, IC9 LM337, U1 LME49830, U2 LME49830, U8 LME49830

Commit message: Updated schematic, added corrections doc to block diagram.
Parts:
- removed C28, C30, C32, C34: 100uF, rcl:E2,5-6
- removed IC8: LM317MABDTRK, v-reg:DPACK
- removed IC9: LM337, Amplifier_Parts:LM337
- removed R40, R41, R42, R93: (no value), rcl:0204V
- added U$22: MOLEX_6P, Amplifier_Parts:MOLEX_6P
- moved R39 305.8 mm to (-166.4, -894.1)
Connections:
- removed net N$10 (its old number): IC8.1, R39.1, R40.2
- new net N$106: N_S1.PAD, R65.1
- new net N$108: R1.1, U$22.P$5
- new net N$109: N_S2.PAD, R80.1
- new net N$110: N_S.PAD, R50.1
- new net N$64: IC10.7, R39.2, R69.2, U$19.1_2, U$19.1_3
- net +12V: now also U$22.P$1; no longer C28.+, IC8.4, R39.2
- net -12V: now also U$22.P$6; no longer C30.-, IC9.3, R41.2
- net GND: now also U$22.P$4; no longer C28.-, C30.+, C32.-, C34.+, R40.1, R42.1
- net N$105: now also U$22.P$2; no longer R84.2, R91.2, R92.2, R93.1
- net N$26: now also R2.1, U$22.P$3; no longer IC9.1, R41.1, R42.2
- net N$38: now also R39.1, R84.2, R91.2, R92.2; no longer IC10.7, R69.2, R93.2, U$19.1_2, U$19.1_3
- net N$75: no longer N_S.PAD, R50.1
- net N$76: no longer N_S1.PAD, R65.1
- net N$96: no longer N_S2.PAD, R80.1
- net V+: no longer C32.+, IC8.3
- net V-: no longer C34.-, IC9.4

Commit message: added data sheets for connectors and updated schematic
Parts:
- removed R49, R50, R64, R65, R79, R80: 0.1, rcl:0204V
- added PR1, PR2, PR3, PR4, PR5, PR6: 0.1, Power Resistors:2-1623788-1
Connections:
- net N$106: now also PR2.P$3; no longer R65.1
- net N$109: now also PR6.P$3; no longer R80.1
- net N$110: now also PR3.P$3; no longer R50.1
- net N$71: now also PR1.P$4; no longer R64.2
- net N$74: now also PR4.P$4; no longer R49.2
- net N$75: now also PR3.P$4, PR4.P$3; no longer R49.1, R50.2
- net N$76: now also PR1.P$3, PR2.P$4; no longer R64.1, R65.2
- net N$95: now also PR5.P$4; no longer R79.2
- net N$96: now also PR5.P$3, PR6.P$4; no longer R79.1, R80.2
Changed lines of the file:
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@@
 <element name="N_S" library="Amplifier_Parts" package="SMT_PAD_5MM" value="SMT_PAD_5MM" x="-100.33" y="-118.11"/>
 <element name="N_D" library="Amplifier_Parts" package="SMT_PAD_5MM" value="SMT_PAD_5MM" x="-100.33" y="-124.46"/>
-<element name="R49" library="rcl" package="0204V" value="0.1" x="-99.06" y="-130.81"/>
-<element name="R50" library="rcl" package="0204V" value="0.1" x="-99.06" y="-135.89"/>
 <element name="C22" library="rcl" package="E2,5-6" value="100uF" x="-100.33" y="-140.97"/>
 <element name="C23" library="rcl" package="E2,5-6" value="100uF" x="-100.33" y="-148.59"/>
@@
 <element name="N_S1" library="Amplifier_Parts" package="SMT_PAD_5MM" value="SMT_PAD_5MM" x="-152.4" y="-735.33"/>
 <element name="N_D1" library="Amplifier_Parts" package="SMT_PAD_5MM" value="SMT_PAD_5MM" x="-119.38" y="-728.98"/>
-<element name="R64" library="rcl" package="0204V" value="0.1" x="-125.73" y="-722.63"/>
-<element name="R65" library="rcl" package="0204V" value="0.1" x="-120.65" y="-722.63"/>
 <element name="C57" library="rcl" package="E2,5-6" value="100uF" x="-151.13" y="-702.31"/>
 <element name="C58" library="rcl" package="E2,5-6" value="100uF" x="-138.43" y="-702.31"/>
@@
 <element name="N_S2" library="Amplifier_Parts" package="SMT_PAD_5MM" value="SMT_PAD_5MM" x="-152.4" y="-788.67"/>
 <element name="N_D2" library="Amplifier_Parts" package="SMT_PAD_5MM" value="SMT_PAD_5MM" x="-119.38" y="-782.32"/>
-<element name="R79" library="rcl" package="0204V" value="0.1" x="-125.73" y="-775.97"/>
-<element name="R80" library="rcl" package="0204V" value="0.1" x="-120.65" y="-775.97"/>
 <element name="C72" library="rcl" package="E2,5-6" value="100uF" x="-151.13" y="-755.65"/>
 <element name="C73" library="rcl" package="E2,5-6" value="100uF" x="-138.43" y="-755.65"/>
@@
 <element name="U$22" library="Amplifier_Parts" package="MOLEX_6P" value="MOLEX_6P" x="-165.1" y="-881.38"/>
 <element name="R39" library="rcl" package="0204V" value="" x="-166.37" y="-894.08"/>
+<element name="PR1" library="Power Resistors" package="2-1623788-1" value="0.1" x="-177.8" y="-890.27">
+<attribute name="MAX_POWER" value="5W" x="-177.8" y="-890.27" size="1.778" layer="27" display="off"/>
+<attribute name="POWER_LEVEL" value="5W" x="-177.8" y="-890.27" size="1.778" layer="27" display="off"/>
+</element>
+<element name="PR2" library="Power Resistors" package="2-1623788-1" value="0.1" x="-191.77" y="-890.27">
+<attribute name="POWER_LEVEL" value="5W" x="-191.77" y="-890.27" size="1.778" layer="27" display="off"/>
+</element>
+<element name="PR3" library="Power Resistors" package="2-1623788-1" value="0.1" x="-205.74" y="-890.27">
+<attribute name="POWER_LEVEL" value="5W" x="-205.74" y="-890.27" size="1.778" layer="27" display="off"/>
+<attribute name="MAX_POWER" value="5W" x="-205.74" y="-890.27" size="1.778" layer="27" display="off"/>
+</element>
+<element name="PR4" library="Power Resistors" package="2-1623788-1" value="0.1" x="-219.71" y="-890.27">
+<attribute name="POWER_LEVEL" value="5W" x="-219.71" y="-890.27" size="1.778" layer="27" display="off"/>
+<attribute name="MAX_POWER" value="5W" x="-219.71" y="-890.27" size="1.778" layer="27" display="off"/>
+</element>
+<element name="PR5" library="Power Resistors" package="2-1623788-1" value="0.1" x="-233.68" y="-890.27">
+<attribute name="POWER_LEVEL" value="5W" x="-233.68" y="-890.27" size="1.778" layer="27" display="off"/>
+</element>
+<element name="PR6" library="Power Resistors" package="2-1623788-1" value="0.1" x="-247.65" y="-890.27">
+<attribute name="POWER_LEVEL" value="5W" x="-247.65" y="-890.27" size="1.778" layer="27" display="off"/>
+</element>
 </elements>
 <signals>
@@
 <signal name="N$74">
 <contactref element="P_S" pad="PAD"/>
-<contactref element="R49" pad="2"/>
-<wire x1="-100.33" y1="-105.41" x2="-97.79" y2="-130.81" width="0" layer="19" extent="1-1"/>
+<contactref element="PR4" pad="P$4"/>
+<wire x1="-217.21" y1="-890.27" x2="-100.33" y2="-105.41" width="0" layer="19" extent="1-1"/>
 </signal>
 <signal name="N$75">
-<contactref element="R50" pad="2"/>
-<contactref element="R49" pad="1"/>
 <contactref element="R51" pad="2"/>
 <contactref element="U8" pad="8"/>
 <contactref element="R56" pad="1"/>
 <contactref element="U$17" pad="P$1"/>
-<wire x1="-100.33" y1="-130.81" x2="-97.79" y2="-135.89" width="0" layer="19" extent="1-1"/>
-<wire x1="-97.79" y1="-167.64" x2="-97.79" y2="-135.89" width="0" layer="19" extent="1-1"/>
-<wire x1="-87.225" y1="-2.54" x2="-100.33" y2="-130.81" width="0" layer="19" extent="1-1"/>
-<wire x1="-143.41" y1="-677.03" x2="-97.79" y2="-167.64" width="0" layer="19" extent="1-1"/>
-<wire x1="-130.81" y1="-685.8" x2="-143.41" y2="-677.03" width="0" layer="19" extent="1-1"/>
+<contactref element="PR3" pad="P$4"/>
+<contactref element="PR4" pad="P$3"/>
+<wire x1="-203.24" y1="-890.27" x2="-222.21" y2="-890.27" width="0" layer="19" extent="1-1"/>
+<wire x1="-130.81" y1="-685.8" x2="-203.24" y2="-890.27" width="0" layer="19" extent="1-1"/>
+<wire x1="-143.41" y1="-677.03" x2="-130.81" y2="-685.8" width="0" layer="19" extent="1-1"/>
+<wire x1="-97.79" y1="-167.64" x2="-143.41" y2="-677.03" width="0" layer="19" extent="1-1"/>
+<wire x1="-87.225" y1="-2.54" x2="-97.79" y2="-167.64" width="0" layer="19" extent="1-1"/>
 </signal>
 <signal name="N$84">
@@
 <signal name="N$71">
 <contactref element="P_S1" pad="PAD"/>
-<contactref element="R64" pad="2"/>
-<wire x1="-124.46" y1="-722.63" x2="-133.35" y2="-735.33" width="0" layer="19" extent="1-1"/>
+<contactref element="PR1" pad="P$4"/>
+<wire x1="-175.3" y1="-890.27" x2="-133.35" y2="-735.33" width="0" layer="19" extent="1-1"/>
 </signal>
 <signal name="N$76">
-<contactref element="R65" pad="2"/>
-<contactref element="R64" pad="1"/>
 <contactref element="R66" pad="2"/>
 <contactref element="U1" pad="8"/>
 <contactref element="R71" pad="1"/>
 <contactref element="U$17" pad="P$3"/>
-<wire x1="-127" y1="-722.63" x2="-132.08" y2="-728.98" width="0" layer="19" extent="1-1"/>
-<wire x1="-119.38" y1="-722.63" x2="-127" y2="-722.63" width="0" layer="19" extent="1-1"/>
-<wire x1="-114.3" y1="-722.63" x2="-119.38" y2="-722.63" width="0" layer="19" extent="1-1"/>
-<wire x1="-146.915" y1="-708.66" x2="-127" y2="-722.63" width="0" layer="19" extent="1-1"/>
+<contactref element="PR1" pad="P$3"/>
+<contactref element="PR2" pad="P$4"/>
+<wire x1="-114.3" y1="-722.63" x2="-132.08" y2="-728.98" width="0" layer="19" extent="1-1"/>
+<wire x1="-146.915" y1="-708.66" x2="-132.08" y2="-728.98" width="0" layer="19" extent="1-1"/>
 <wire x1="-147.71" y1="-677.03" x2="-146.915" y2="-708.66" width="0" layer="19" extent="1-1"/>
+<wire x1="-180.3" y1="-890.27" x2="-132.08" y2="-728.98" width="0" layer="19" extent="1-1"/>
+<wire x1="-189.27" y1="-890.27" x2="-180.3" y2="-890.27" width="0" layer="19" extent="1-1"/>
 </signal>
 <signal name="N$77">
@@
 <signal name="N$95">
 <contactref element="P_S2" pad="PAD"/>
-<contactref element="R79" pad="2"/>
-<wire x1="-124.46" y1="-775.97" x2="-133.35" y2="-788.67" width="0" layer="19" extent="1-1"/>
+<contactref element="PR5" pad="P$4"/>
+<wire x1="-231.18" y1="-890.27" x2="-133.35" y2="-788.67" width="0" layer="19" extent="1-1"/>
 </signal>
 <signal name="N$96">
-<contactref element="R80" pad="2"/>
-<contactref element="R79" pad="1"/>
 <contactref element="R81" pad="2"/>
 <contactref element="U2" pad="8"/>
 <contactref element="R86" pad="1"/>
 <contactref element="U$17" pad="P$5"/>
-<wire x1="-127" y1="-775.97" x2="-132.08" y2="-782.32" width="0" layer="19" extent="1-1"/>
-<wire x1="-119.38" y1="-775.97" x2="-127" y2="-775.97" width="0" layer="19" extent="1-1"/>
-<wire x1="-114.3" y1="-775.97" x2="-119.38" y2="-775.97" width="0" layer="19" extent="1-1"/>
-<wire x1="-146.915" y1="-762" x2="-127" y2="-775.97" width="0" layer="19" extent="1-1"/>
+<contactref element="PR5" pad="P$3"/>
+<contactref element="PR6" pad="P$4"/>
+<wire x1="-114.3" y1="-775.97" x2="-132.08" y2="-782.32" width="0" layer="19" extent="1-1"/>
+<wire x1="-146.915" y1="-762" x2="-132.08" y2="-782.32" width="0" layer="19" extent="1-1"/>
 <wire x1="-147.71" y1="-671.33" x2="-146.915" y2="-762" width="0" layer="19" extent="1-1"/>
+<wire x1="-236.18" y1="-890.27" x2="-132.08" y2="-782.32" width="0" layer="19" extent="1-1"/>
+<wire x1="-245.15" y1="-890.27" x2="-236.18" y2="-890.27" width="0" layer="19" extent="1-1"/>
 </signal>
 <signal name="N$97">
@@
 </signal>
 <signal name="N$106">
-<contactref element="R65" pad="1"/>
 <contactref element="N_S1" pad="PAD"/>
-<wire x1="-121.92" y1="-722.63" x2="-152.4" y2="-735.33" width="0" layer="19" extent="1-1"/>
+<contactref element="PR2" pad="P$3"/>
+<wire x1="-194.27" y1="-890.27" x2="-152.4" y2="-735.33" width="0" layer="19" extent="1-1"/>
 </signal>
 <signal name="N$109">
 <contactref element="N_S2" pad="PAD"/>
-<contactref element="R80" pad="1"/>
-<wire x1="-121.92" y1="-775.97" x2="-152.4" y2="-788.67" width="0" layer="19" extent="1-1"/>
+<contactref element="PR6" pad="P$3"/>
+<wire x1="-250.15" y1="-890.27" x2="-152.4" y2="-788.67" width="0" layer="19" extent="1-1"/>
 </signal>
 <signal name="N$110">
 <contactref element="N_S" pad="PAD"/>
-<contactref element="R50" pad="1"/>
-<wire x1="-100.33" y1="-118.11" x2="-100.33" y2="-135.89" width="0" layer="19" extent="1-1"/>
+<contactref element="PR3" pad="P$3"/>
+<wire x1="-208.24" y1="-890.27" x2="-100.33" y2="-118.11" width="0" layer="19" extent="1-1"/>
 </signal>
 </signals>
