File: Schematics/Audio _Eagle/Amplifier_v1.1.sch (EAGLE design)
At the start: 100 parts, among them U1 NE5532, U2 NE5532, U3 NE5532, U4 NE5532, U5 NE5532, U6 NE5532, U7 NE5532, U8 LME49830

Commit message: update to amp schematic
Parts:
- removed R39: (no value), resistor:R-US_0207/7
- removed R40, R41, R42: (no value), pot:3RP/1610G
- removed U1, U2, U3, U4, U5, U6, U7: NE5532, NE5532:NE5532
- added C22, C23, C27: 100uF, rcl:CPOL-USE2.5-6
- added C24, C25, C26: 0.1uF, rcl:C-EU025-024X044
- added C29, C31, C33, C35, C37, C39, C41, C43, C45, C47, C49, C51, C53, C55: 10uF, rcl:C-EU025-024X044
- added IC1, IC2, IC3, IC4, IC5, IC6, IC7: NE5532N, linear:NE5532N
- added R51: 10, rcl:R-US_0204/2V
- added R52: 1.2k, rcl:R-US_0204/2V
- added U$13, U$14: TONE_POT_2GANG, Amplifier_Parts:TONE_POT_2GANG
- added U$15: INDUCTOR, Amplifier_Parts:INDUCTOR
- added U$16: VOL_POT_2GANG, Amplifier_Parts:VOL_POT_2GANG
- R1, R10, R11, R12, R13, R14, R15, R16, R17, R18, R19, R2, R20, R21, R22, R23, R24, R25, R26, R27, R28, R29, R30, R31, R32, R33, R34, R35, R36, R37, R38, R4, R44, R45, R47, R48, R49, R5, R50, R6, R7, R8, R9: device resistor:R-US_0207/7 -> rcl:R-US_0204/2V
- R3: device pot:3RP/1610G -> rcl:R-US_0204/2V
- R46: value 1.2k -> 12k; device resistor:R-US_0207/7 -> rcl:R-US_0204/2V
- U$1: value INDUCTOR -> TONE_POT_2GANG; device Amplifier_Parts:INDUCTOR -> Amplifier_Parts:TONE_POT_2GANG
Connections:
- removed net N$10: R6.1, R8.2, U2G$1.P$3
- removed net N$16: C7.2, C8.2, U$5.1
- removed net N$20: R10.1, U$3.1, U$4.1
- removed net N$26: R16.2, R36.1, U4G$2.P$1
- removed net N$28: R15.1, U$6.1
- removed net N$31: C10.1, C11.1, R20.1
- removed net N$36: C12.2, R24.2, U$8.2
- removed net N$39: R26.1, R27.2, U6G$1.P$3
- removed net N$4: C10.2, R19.2, U$1.1
- removed net N$40: R26.2, R38.1, U6G$2.P$1
- removed net N$48: U7G$2.P$2
- removed net N$51: C13.1, U$12.1
- removed net N$52: C9.2, R19.1, R24.1, R29.1
- removed net N$62: R38.2, R41/2.A
- removed net N$63 (its old number): R42/2.E, R42/2.S, U7G$2.P$3
- removed net N$8: C3.1, C4.1, R5.1
- new net GND: C10.1, C11.1, C14.2, C15.2, C16.-, C17.1, C18.2, C2.+, C22.-, C23.+, C24.2, C25.1, C26.1, C27.-, C29.1, C3.1, C31.2, C33.1, C35.2, C37.1, C39.2, C4.1, C41.1, C43.2, C45.1, C47.2, C49.1, C51.2, C53.1, C55.2, C7.2, C8.2, IC1B.+IN, IC2B.+IN, IC3B.+IN, IC4B.+IN, IC5B.+IN, IC6B.+IN, IC7A.+IN, IC7B.+IN, R10.1, R13.1, R15.1, R20.1, R23.1, R26.1, R28.1, R3.2, R31.2, R38.1, R5.1, R7.1, U$10.1, U$11.1, U$12.1, U$3.1, U$4.1, U$5.1, U$6.1, U$9.1
- new net N$30: IC4B.-IN, R19.2, R29.1
- new net N$80: C17.2, C2.-, U8.-VEE
- new net N$82: C16.+, C18.1, U8.+VCC
- new net N$84: C26.2, R51.1
- new net N$85: C27.+, R52.2, U8.MUTE
- new net N$88: IC1A.OUT, R6.1, R8.2
- new net VCC: C22.+, C24.1, C31.1, C35.1, C39.1, C43.1, C47.1, C51.1, C55.1, IC1P.V+, IC2P.V+, IC3P.V+, IC4P.V+, IC5P.V+, IC6P.V+, IC7P.V+, P_D.PAD
- new net VEE: C23.-, C25.2, C29.2, C33.2, C37.2, C41.2, C45.2, C49.2, C53.2, IC1P.V-, IC2P.V-, IC3P.V-, IC4P.V-, IC5P.V-, IC6P.V-, IC7P.V-, N_D.PAD
- net N$1: now also IC7A.-IN, U$16G$1.1_1; no longer R3/2.A, U1G$1.P$1
- net N$11: now also IC1B.-IN; no longer U2G$2.P$1
- net N$12: now also C3.2, IC1A.+IN, R3.1, U$2.1; no longer U2G$2.P$2
- net N$14: now also IC2A.+IN; no longer U3G$1.P$2
- net N$15: now also IC3A.OUT, R16.1, R17.2; no longer R12.1, R13.2, U3G$1.P$1
- net N$17: now also IC2A.OUT; no longer U3G$1.P$3
- net N$18: now also IC2B.-IN; no longer U3G$2.P$1
- net N$19: now also IC3B.-IN, R16.2, R18.1; no longer U3G$2.P$2
- net N$2: now also IC7A.OUT, U$16G$1.1_2, U$16G$1.1_3; no longer R3/2.E, R3/2.S, U1G$1.P$3
- net N$21: now also IC3B.OUT, U$14G$1.1_2, U$14G$1.1_3; no longer C11.2, R20.2, U$1.2, U5G$1.P$2
- net N$23: now also IC3A.+IN; no longer U4G$1.P$2
- net N$24: now also U$14G$1.1_1; no longer R17.1, U4G$1.P$1
- net N$25: now also C11.2, R32.2, U$8.2; no longer R16.1, R17.2, U4G$1.P$3
- net N$27: now also IC3A.-IN, R17.1, R5.2; no longer U4G$2.P$2
- net N$3: now also IC7B.-IN, U$16G$2.1_1; no longer R3/1.A, U1G$2.P$1
- net N$32: now also C12.2, U$9.2; no longer R23.1, U5G$1.P$1
- net N$33: now also C12.1, IC5A.+IN, U$10.2; no longer R21.1, U5G$1.P$3
- net N$34: now also IC5A.OUT, R24.1, R25.2; no longer R21.2, R37.1, U5G$2.P$1
- net N$35: now also IC5B.-IN, R24.2, R30.1; no longer U5G$2.P$2
- net N$37: now also C13.2, C15.1, R27.2, U$11.2; no longer C12.1, R25.2, U$9.2, U6G$1.P$2
- net N$38: now also C14.1, IC6A.+IN, U$12.2, U$15.2; no longer R27.1, U6G$1.P$1
- net N$41: now also C13.1, U$15.1; no longer U6G$2.P$2
- net N$42: now also R29.2, U$1G$2.1_1; no longer R25.1, U$8.1, U$9.1
- net N$43: now also IC4B.OUT, U$1G$2.1_2, U$1G$2.1_3; no longer C13.2, C15.1, R29.2, U$10.2
- net N$44: now also IC5B.OUT, U$13G$2.1_2, U$13G$2.1_3; no longer C14.1, R30.2, U$11.2, U$12.2, U7G$1.P$2
- net N$45: now also R30.2, U$13G$2.1_1; no longer R32.1, R33.2, U7G$1.P$1
- net N$46: now also IC4A.OUT, R19.1, R21.2; no longer R31.1, R32.2, U7G$1.P$3
- net N$47: now also C10.2, IC4A.+IN, R31.1, U$8.1; no longer R31.2, R39.1, U7G$2.P$1
- net N$49: now also IC4A.-IN, R20.2, R21.1; no longer R30.1, U$11.1
- net N$5: now also IC7B.OUT, U$16G$2.1_2, U$16G$2.1_3; no longer R3/1.E, R3/1.S, U1G$2.P$3
- net N$50: now also IC5A.-IN, R25.1, R26.2; no longer C14.2, C15.2, U$10.1
- net N$53: now also U$1G$1.1_1; no longer R40/1.A
- net N$54: now also IC1B.OUT, U$1G$1.1_2, U$1G$1.1_3; no longer R40/1.E, R40/1.S, U2G$2.P$3
- net N$55: now also IC2B.OUT, U$13G$1.1_2, U$13G$1.1_3; no longer R41/1.E, R41/1.S, U3G$2.P$3
- net N$56: now also U$13G$1.1_1; no longer R41/1.A
- net N$57: now also IC6A.OUT, R33.1, R36.2; no longer R42/1.E, R42/1.S, U4G$2.P$3
- net N$58: now also IC6B.-IN, R33.2, R37.1; no longer R36.2, R42/1.A
- net N$59: now also IC6B.OUT, U$14G$2.1_2, U$14G$2.1_3; no longer R40/2.E, R40/2.S, U5G$2.P$3
- net N$6: now also IC1A.-IN, R7.2, R8.1; no longer C3.2, R4.2, U$2.1
- net N$60: now also U$14G$2.1_1; no longer R40/2.A
- net N$61: now also IC6A.-IN, R36.1, R38.2; no longer R41/2.E, R41/2.S, U6G$2.P$3
- net N$64: now also C9.2, R22.1, R27.1, R32.1; no longer R39.2, R42/2.A
- net N$7: now also R4.2; no longer R5.2, U2G$1.P$2
- net N$74: now also P_S.PAD; no longer P_D.PAD
- net N$75: now also N_S.PAD, R51.2; no longer N_D.PAD
- net N$9: now also IC2A.-IN, R12.1, R13.2; no longer R7.2, R8.1, U2G$1.P$1
Other:
- note added: "MOSFET_n"
- note added: "MOSFET_p"
- note added: "change this footprint to a bigger drill"
- note removed: "BASS LEFT CHANNEL"
- note removed: "MIDS LEFT CHANNEL"
- note removed: "MOSFET_N"
- note removed: "MOSFET_P"
- note removed: "TREBLE LEFT CHANNEL"
- moved on the sheet: C1, C10, C11, C12, C13, C14, C15, C3, C4, C5, C6, C7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

Commit message: updated schematic
Parts:
- added IC8: LM317MABDTRK, v-reg:LM317MABDTRK
- added IC9: LM337, Amplifier_Parts:LM337
- C29, C31, C33, C35, C37, C39, C41, C43, C45, C47, C49, C51, C53, C55: value 10uF -> 0.1uF
Changed lines of the file:
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@@
 <part name="U$13" library="Amplifier_Parts" deviceset="TONE_POT_2GANG" device=""/>
 <part name="U$14" library="Amplifier_Parts" deviceset="TONE_POT_2GANG" device=""/>
-<part name="C29" library="rcl" deviceset="C-EU" device="025-024X044" value="10uF"/>
-<part name="C31" library="rcl" deviceset="C-EU" device="025-024X044" value="10uF"/>
-<part name="C33" library="rcl" deviceset="C-EU" device="025-024X044" value="10uF"/>
-<part name="C35" library="rcl" deviceset="C-EU" device="025-024X044" value="10uF"/>
-<part name="C37" library="rcl" deviceset="C-EU" device="025-024X044" value="10uF"/>
-<part name="C39" library="rcl" deviceset="C-EU" device="025-024X044" value="10uF"/>
-<part name="C41" library="rcl" deviceset="C-EU" device="025-024X044" value="10uF"/>
-<part name="C43" library="rcl" deviceset="C-EU" device="025-024X044" value="10uF"/>
-<part name="C45" library="rcl" deviceset="C-EU" device="025-024X044" value="10uF"/>
-<part name="C47" library="rcl" deviceset="C-EU" device="025-024X044" value="10uF"/>
-<part name="C49" library="rcl" deviceset="C-EU" device="025-024X044" value="10uF"/>
-<part name="C51" library="rcl" deviceset="C-EU" device="025-024X044" value="10uF"/>
-<part name="C53" library="rcl" deviceset="C-EU" device="025-024X044" value="10uF"/>
-<part name="C55" library="rcl" deviceset="C-EU" device="025-024X044" value="10uF"/>
+<part name="C29" library="rcl" deviceset="C-EU" device="025-024X044" value="0.1uF"/>
+<part name="C31" library="rcl" deviceset="C-EU" device="025-024X044" value="0.1uF"/>
+<part name="C33" library="rcl" deviceset="C-EU" device="025-024X044" value="0.1uF"/>
+<part name="C35" library="rcl" deviceset="C-EU" device="025-024X044" value="0.1uF"/>
+<part name="C37" library="rcl" deviceset="C-EU" device="025-024X044" value="0.1uF"/>
+<part name="C39" library="rcl" deviceset="C-EU" device="025-024X044" value="0.1uF"/>
+<part name="C41" library="rcl" deviceset="C-EU" device="025-024X044" value="0.1uF"/>
+<part name="C43" library="rcl" deviceset="C-EU" device="025-024X044" value="0.1uF"/>
+<part name="C45" library="rcl" deviceset="C-EU" device="025-024X044" value="0.1uF"/>
+<part name="C47" library="rcl" deviceset="C-EU" device="025-024X044" value="0.1uF"/>
+<part name="C49" library="rcl" deviceset="C-EU" device="025-024X044" value="0.1uF"/>
+<part name="C51" library="rcl" deviceset="C-EU" device="025-024X044" value="0.1uF"/>
+<part name="C53" library="rcl" deviceset="C-EU" device="025-024X044" value="0.1uF"/>
+<part name="C55" library="rcl" deviceset="C-EU" device="025-024X044" value="0.1uF"/>
 <part name="GND1" library="supply2" deviceset="GND" device=""/>
 <part name="GND2" library="supply2" deviceset="GND" device=""/>
@@
 <part name="SUPPLY4" library="supply2" deviceset="GND" device=""/>
 <part name="GND16" library="supply2" deviceset="GND" device=""/>
+<part name="IC8" library="v-reg" deviceset="LM317?*" device="" technology="MABDTRK"/>
+<part name="IC9" library="Amplifier_Parts" deviceset="LM337" device=""/>
 </parts>
 <sheets>
@@
 <instance part="SUPPLY4" gate="GND" x="439.42" y="129.54" rot="R180"/>
 <instance part="GND16" gate="GND" x="124.46" y="40.64"/>
+<instance part="IC8" gate="G$1" x="215.9" y="177.8"/>
+<instance part="IC9" gate="G$1" x="256.54" y="175.26"/>
 </instances>
 <busses>

Commit message: amp schematic updates
Parts:
- added C28, C30, C32, C34, C36, C38: 100uF, rcl:CPOL-USE2.5-6
- added C40, C42: 0.1uF, rcl:C-EU025-024X044
- added R39, R40, R41, R42: (no value), rcl:R-US_0204/2V
- added R53, R54, R55, R56: 1.2k, rcl:R-US_0204/2V
- added R57: (no value), pot:TRIM_EU-B25U
- added U$17: MOLEX_6P, Amplifier_Parts:MOLEX_6P
Connections:
- net N$82 renamed V+
- removed net N$71: R48.2, U8.OSENSE
- removed net N$80: C17.2, C2.-, U8.-VEE
- removed net VEE: C23.-, C25.2, C29.2, C33.2, C37.2, C41.2, C45.2, C49.2, C53.2, IC1P.V-, IC2P.V-, IC3P.V-, IC4P.V-, IC5P.V-, IC6P.V-, IC7P.V-, N_D.PAD
- new net +12V: C31.1, C32.+, C35.1, C36.+, C39.1, C43.1, C47.1, C51.1, C55.1, IC1P.V+, IC2P.V+, IC3P.V+, IC4P.V+, IC5P.V+, IC6P.V+, IC7P.V+, IC8.IN
- new net -12V: C29.2, C33.2, C34.-, C37.2, C38.-, C41.2, C45.2, C49.2, C53.2, IC1P.V-, IC2P.V-, IC3P.V-, IC4P.V-, IC5P.V-, IC6P.V-, IC7P.V-, IC9.IN
- new net N$10: IC8.ADJ, R39.1, R40.2
- new net N$16: C40.2, R53.1, R54.1, U8.IN+
- new net N$20: C28.+, IC8.OUT, R39.2
- new net N$26: IC9.ADJ, R41.1, R42.2
- new net N$28: C30.-, IC9.OUT, R41.2
- new net N$31: R55.1, R57.A, U8.IN-
- new net N$36: C42.2, R55.2
- new net N$4: R48.2, U8.N_OUT
- new net N$40: R56.2, R57.E, R57.S
- new net N$8: C22.-, C24.2
- new net V-: C17.2, C2.-, C23.-, C25.2, N_D.PAD, U8.-VEE
- net GND: now also C28.-, C30.+, C32.-, C34.+, C36.-, C38.+, C40.1, C42.1, R40.1, R42.1, R53.2, U$17.S1, U8.GND; no longer C22.-, C24.2
- net N$68: now also R43.S
- net N$75: now also R56.1, U$17.S, U8.OSENSE
- net VCC: no longer C31.1, C35.1, C39.1, C43.1, C47.1, C51.1, C55.1, IC1P.V+, IC2P.V+, IC3P.V+, IC4P.V+, IC5P.V+, IC6P.V+, IC7P.V+
Other:
- note added: "change footprint"
- note added: "the foot print need to change"
- note removed: "change this footprint to a bigger drill"
- moved on the sheet: C16, C17, C18, C2, C26, IC9

Commit message: updated schematic
Connections:
- removed net N$20: C28.+, IC8.OUT, R39.2
- removed net N$28: C30.-, IC9.OUT, R41.2
- removed net N$8: C22.-, C24.2
- net +12V: now also C28.+, IC8.OUT, R39.2; no longer C32.+, IC8.IN
- net -12V: now also C30.-, IC9.OUT, R41.2; no longer C34.-, IC9.IN
- net GND: now also C22.-, C24.2
- net V+: now also C32.+, IC8.IN
- net V-: now also C34.-, IC9.IN
Other:
- moved on the sheet: B_R_B, B_R_C, B_R_E, C1, C10, C11, C12, C13, C14, C15, C16, C17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
