File: Schematics/Audio _Eagle/Amplifier_v1.1.sch (EAGLE design)
At the start: 236 parts, among them IC1 NE5532N, IC10 NE5532N, IC11 NE5532N, IC12 NE5532N, IC13 NE5532N, IC2 NE5532N, IC3 NE5532N, IC4 NE5532N, IC5 NE5532N, IC6 NE5532N, IC7 NE5532N, IC8 LM317MABDTRK, IC9 LM337, U1 LME49830, U2 LME49830, U8 LME49830

Commit message: Updated schematic, added corrections doc to block diagram.
Parts:
- removed C28, C30, C32, C34: 100uF, rcl:CPOL-USE2.5-6
- removed IC8: LM317MABDTRK, v-reg:LM317MABDTRK
- removed IC9: LM337, Amplifier_Parts:LM337
- removed R40, R41, R42, R93: (no value), rcl:R-US_0204/2V
- added U$22: MOLEX_6P, Amplifier_Parts:MOLEX_6P
Connections:
- removed net N$10 (its old number): IC8.ADJ, R39.1, R40.2
- new net N$106: N_S1.PAD, R65.1
- new net N$108: R1.1, U$22.S4
- new net N$109: N_S2.PAD, R80.1
- new net N$110: N_S.PAD, R50.1
- new net N$64: IC10B.OUT, R39.2, R69.2, U$19G$1.1_2, U$19G$1.1_3
- net +12V: now also U$22.S; no longer C28.+, IC8.OUT, R39.2
- net -12V: now also U$22.S5; no longer C30.-, IC9.OUT, R41.2
- net GND: now also U$22.S3; no longer C28.-, C30.+, C32.-, C34.+, R40.1, R42.1
- net N$105: now also U$22.S1; no longer R84.2, R91.2, R92.2, R93.1
- net N$26: now also R2.1, U$22.S2; no longer IC9.ADJ, R41.1, R42.2
- net N$38: now also R39.1, R84.2, R91.2, R92.2; no longer IC10B.OUT, R69.2, R93.2, U$19G$1.1_2, U$19G$1.1_3
- net N$75: no longer N_S.PAD, R50.1
- net N$76: no longer N_S1.PAD, R65.1
- net N$96: no longer N_S2.PAD, R80.1
- net V+: no longer C32.+, IC8.IN
- net V-: no longer C34.-, IC9.IN
Other:
- note added: "Left"
- note added: "Mute"
- note added: "Right"
- note added: "altleast .5W"
- moved on the sheet: C17, IC12A, IC7A, R1, R2, R39, U$16G$1, U$18G$1

Commit message: added data sheets for connectors and updated schematic
Parts:
- removed R49, R50, R64, R65, R79, R80: 0.1, rcl:R-US_0204/2V
- added P1: 18AWG, AWG Holes:18AWG
- added PR1, PR2, PR3, PR4, PR5, PR6: (no value), Power Resistors:SQM
Connections:
- net N$106: now also PR3.1; no longer R65.1
- net N$109: now also PR2.1; no longer R80.1
- net N$110: now also PR5.1; no longer R50.1
- net N$71: now also PR4.2; no longer R64.2
- net N$74: now also PR6.2; no longer R49.2
- net N$75: now also PR5.2, PR6.1; no longer R49.1, R50.2
- net N$76: now also PR3.2, PR4.1; no longer R64.1, R65.2
- net N$95: now also PR1.2; no longer R79.2
- net N$96: now also PR1.1, PR2.2; no longer R79.1, R80.2
Other:
- note removed: "the foot print need to change"
Changed lines of the file:
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@@
 <part name="N_S" library="Amplifier_Parts" deviceset="SMT_PAD_5MM" device=""/>
 <part name="N_D" library="Amplifier_Parts" deviceset="SMT_PAD_5MM" device=""/>
-<part name="R49" library="rcl" deviceset="R-US_" device="0204/2V" value="0.1"/>
-<part name="R50" library="rcl" deviceset="R-US_" device="0204/2V" value="0.1"/>
 <part name="C22" library="rcl" deviceset="CPOL-US" device="E2.5-6" value="100uF"/>
 <part name="C23" library="rcl" deviceset="CPOL-US" device="E2.5-6" value="100uF"/>
@@
 <part name="N_S1" library="Amplifier_Parts" deviceset="SMT_PAD_5MM" device=""/>
 <part name="N_D1" library="Amplifier_Parts" deviceset="SMT_PAD_5MM" device=""/>
-<part name="R64" library="rcl" deviceset="R-US_" device="0204/2V" value="0.1"/>
-<part name="R65" library="rcl" deviceset="R-US_" device="0204/2V" value="0.1"/>
 <part name="C57" library="rcl" deviceset="CPOL-US" device="E2.5-6" value="100uF"/>
 <part name="C58" library="rcl" deviceset="CPOL-US" device="E2.5-6" value="100uF"/>
@@
 <part name="N_S2" library="Amplifier_Parts" deviceset="SMT_PAD_5MM" device=""/>
 <part name="N_D2" library="Amplifier_Parts" deviceset="SMT_PAD_5MM" device=""/>
-<part name="R79" library="rcl" deviceset="R-US_" device="0204/2V" value="0.1"/>
-<part name="R80" library="rcl" deviceset="R-US_" device="0204/2V" value="0.1"/>
 <part name="C72" library="rcl" deviceset="CPOL-US" device="E2.5-6" value="100uF"/>
 <part name="C73" library="rcl" deviceset="CPOL-US" device="E2.5-6" value="100uF"/>
@@
 <part name="P-1" library="supply1" deviceset="-12V" device=""/>
 <part name="R39" library="rcl" deviceset="R-US_" device="0204/2V"/>
+<part name="PR1" library="Power Resistors" deviceset="SQM" device=""/>
+<part name="PR2" library="Power Resistors" deviceset="SQM" device=""/>
+<part name="PR3" library="Power Resistors" deviceset="SQM" device=""/>
+<part name="PR4" library="Power Resistors" deviceset="SQM" device=""/>
+<part name="PR5" library="Power Resistors" deviceset="SQM" device=""/>
+<part name="PR6" library="Power Resistors" deviceset="SQM" device=""/>
+<part name="P1" library="AWG Holes" deviceset="18AWG" device=""/>
 </parts>
 <sheets>
@@
 <text x="500.38" y="259.08" size="1.778" layer="97">change
 footprint</text>
-<text x="482.6" y="274.32" size="1.778" layer="97">the foot print
-need to change</text>
 <text x="444.5" y="139.7" size="1.778" layer="97">Vbe multiplier</text>
 <text x="485.14" y="149.86" size="1.778" layer="97">MOSFET_n</text>
@@
 <text x="500.38" y="119.38" size="1.778" layer="97">change
 footprint</text>
-<text x="482.6" y="134.62" size="1.778" layer="97">the foot print
-need to change</text>
 <text x="444.5" y="20.32" size="1.778" layer="97">Vbe multiplier</text>
 <text x="485.14" y="30.48" size="1.778" layer="97">MOSFET_n</text>
@@
 <text x="500.38" y="0" size="1.778" layer="97">change
 footprint</text>
-<text x="482.6" y="15.24" size="1.778" layer="97">the foot print
-need to change</text>
 <text x="464.82" y="335.28" size="6.4516" layer="97">Right Amp</text>
 <text x="462.28" y="198.12" size="6.4516" layer="97">Bass Amp</text>
@@
 <text x="500.38" y="5.08" size="1.778" layer="97">altleast .5W</text>
 <text x="25.4" y="137.16" size="1.778" layer="97">Mute</text>
+<wire x1="93.98" y1="185.42" x2="71.12" y2="170.18" width="0.1524" layer="97" style="shortdash"/>
+<wire x1="71.12" y1="170.18" x2="71.12" y2="43.18" width="0.1524" layer="97" style="shortdash"/>
+<wire x1="71.12" y1="43.18" x2="93.98" y2="58.42" width="0.1524" layer="97" style="shortdash"/>
 </plain>
 <instances>
@@
 <instance part="N_S" gate="G$1" x="480.06" y="251.46" rot="R180"/>
 <instance part="N_D" gate="G$1" x="480.06" y="241.3" rot="R180"/>
-<instance part="R49" gate="G$1" x="477.52" y="276.86" rot="R90"/>
-<instance part="R50" gate="G$1" x="477.52" y="264.16" rot="R90"/>
 <instance part="C22" gate="G$1" x="469.9" y="299.72" rot="R180"/>
 <instance part="C23" gate="G$1" x="469.9" y="236.22" rot="R180"/>
@@
 <instance part="N_S1" gate="G$1" x="480.06" y="111.76" rot="R180"/>
 <instance part="N_D1" gate="G$1" x="480.06" y="101.6" rot="R180"/>
-<instance part="R64" gate="G$1" x="477.52" y="137.16" rot="R90"/>
-<instance part="R65" gate="G$1" x="477.52" y="124.46" rot="R90"/>
 <instance part="C57" gate="G$1" x="469.9" y="160.02" rot="R180"/>
 <instance part="C58" gate="G$1" x="469.9" y="96.52" rot="R180"/>
@@
 <instance part="N_S2" gate="G$1" x="480.06" y="-7.62" rot="R180"/>
 <instance part="N_D2" gate="G$1" x="480.06" y="-17.78" rot="R180"/>
-<instance part="R79" gate="G$1" x="477.52" y="17.78" rot="R90"/>
-<instance part="R80" gate="G$1" x="477.52" y="5.08" rot="R90"/>
 <instance part="C72" gate="G$1" x="469.9" y="40.64" rot="R180"/>
 <instance part="C73" gate="G$1" x="469.9" y="-22.86" rot="R180"/>
@@
 <instance part="P-1" gate="1" x="43.18" y="109.22"/>
 <instance part="R39" gate="G$1" x="304.8" y="73.66" rot="R90"/>
+<instance part="PR1" gate="G$1" x="477.52" y="17.78" rot="R90"/>
+<instance part="PR2" gate="G$1" x="477.52" y="5.08" rot="R90"/>
+<instance part="PR3" gate="G$1" x="477.52" y="124.46" rot="R90"/>
+<instance part="PR4" gate="G$1" x="477.52" y="137.16" rot="R90"/>
+<instance part="PR5" gate="G$1" x="477.52" y="264.16" rot="R90"/>
+<instance part="PR6" gate="G$1" x="477.52" y="276.86" rot="R90"/>
+<instance part="P1" gate="G$1" x="454.66" y="25.4"/>
 </instances>
 <busses>
@@
 <segment>
 <pinref part="P_S" gate="G$1" pin="PAD"/>
-<pinref part="R49" gate="G$1" pin="2"/>
 <wire x1="477.52" y1="287.02" x2="477.52" y2="281.94" width="0.1524" layer="91"/>
+<pinref part="PR6" gate="G$1" pin="2"/>
 </segment>
 </net>
 <net name="N$75" class="0">
 <segment>
-<pinref part="R50" gate="G$1" pin="2"/>
-<pinref part="R49" gate="G$1" pin="1"/>
 <wire x1="477.52" y1="269.24" x2="477.52" y2="271.78" width="0.1524" layer="91"/>
 <pinref part="R51" gate="G$1" pin="2"/>
 <wire x1="495.3" y1="269.24" x2="477.52" y2="269.24" width="0.1524" layer="91"/>
-<junction x="477.52" y="269.24"/>
 <wire x1="508" y1="317.5" x2="508" y2="269.24" width="0.1524" layer="91"/>
 <wire x1="508" y1="269.24" x2="495.3" y2="269.24" width="0.1524" layer="91"/>
@@
 <wire x1="581.66" y1="269.24" x2="508" y2="269.24" width="0.1524" layer="91"/>
 <junction x="508" y="269.24"/>
+<pinref part="PR5" gate="G$1" pin="2"/>
+<junction x="477.52" y="269.24"/>
+<pinref part="PR6" gate="G$1" pin="1"/>
 </segment>
 </net>
@@
 <segment>
 <pinref part="P_S1" gate="G$1" pin="PAD"/>
-<pinref part="R64" gate="G$1" pin="2"/>
 <wire x1="477.52" y1="147.32" x2="477.52" y2="142.24" width="0.1524" layer="91"/>
+<pinref part="PR4" gate="G$1" pin="2"/>
 </segment>
 </net>
 <net name="N$76" class="0">
 <segment>
-<pinref part="R65" gate="G$1" pin="2"/>
-<pinref part="R64" gate="G$1" pin="1"/>
 <wire x1="477.52" y1="129.54" x2="477.52" y2="132.08" width="0.1524" layer="91"/>
 <pinref part="R66" gate="G$1" pin="2"/>
 <wire x1="495.3" y1="129.54" x2="477.52" y2="129.54" width="0.1524" layer="91"/>
-<junction x="477.52" y="129.54"/>
 <wire x1="508" y1="177.8" x2="508" y2="129.54" width="0.1524" layer="91"/>
 <wire x1="508" y1="129.54" x2="495.3" y2="129.54" width="0.1524" layer="91"/>
@@
 <wire x1="581.66" y1="259.08" x2="520.7" y2="259.08" width="0.1524" layer="91"/>
 <wire x1="520.7" y1="259.08" x2="520.7" y2="129.54" width="0.1524" layer="91"/>
+<pinref part="PR3" gate="G$1" pin="2"/>
+<junction x="477.52" y="129.54"/>
+<pinref part="PR4" gate="G$1" pin="1"/>
 </segment>
 </net>
@@
 <segment>
 <pinref part="P_S2" gate="G$1" pin="PAD"/>
-<pinref part="R79" gate="G$1" pin="2"/>
 <wire x1="477.52" y1="27.94" x2="477.52" y2="22.86" width="0.1524" layer="91"/>
+<pinref part="PR1" gate="G$1" pin="2"/>
+<junction x="477.52" y="22.86"/>
 </segment>
 </net>
 <net name="N$96" class="0">
 <segment>
-<pinref part="R80" gate="G$1" pin="2"/>
-<pinref part="R79" gate="G$1" pin="1"/>
 <wire x1="477.52" y1="10.16" x2="477.52" y2="12.7" width="0.1524" layer="91"/>
 <pinref part="R81" gate="G$1" pin="2"/>
 <wire x1="495.3" y1="10.16" x2="477.52" y2="10.16" width="0.1524" layer="91"/>
-<junction x="477.52" y="10.16"/>
 <wire x1="508" y1="58.42" x2="508" y2="10.16" width="0.1524" layer="91"/>
 <wire x1="508" y1="10.16" x2="495.3" y2="10.16" width="0.1524" layer="91"/>
@@
 <pinref part="U$17" gate="G$1" pin="S4"/>
 <wire x1="528.32" y1="248.92" x2="581.66" y2="248.92" width="0.1524" layer="91"/>
+<pinref part="PR2" gate="G$1" pin="2"/>
+<junction x="477.52" y="10.16"/>
+<pinref part="PR1" gate="G$1" pin="1"/>
 </segment>
 </net>
@@
 <segment>
 <pinref part="N_S1" gate="G$1" pin="PAD"/>
-<pinref part="R65" gate="G$1" pin="1"/>
 <wire x1="477.52" y1="119.38" x2="477.52" y2="111.76" width="0.1524" layer="91"/>
+<pinref part="PR3" gate="G$1" pin="1"/>
 </segment>
 </net>
@@
 <segment>
 <pinref part="N_S2" gate="G$1" pin="PAD"/>
-<pinref part="R80" gate="G$1" pin="1"/>
 <wire x1="477.52" y1="0" x2="477.52" y2="-7.62" width="0.1524" layer="91"/>
+<pinref part="PR2" gate="G$1" pin="1"/>
 </segment>
 </net>
@@
 <segment>
 <pinref part="N_S" gate="G$1" pin="PAD"/>
-<pinref part="R50" gate="G$1" pin="1"/>
 <wire x1="477.52" y1="259.08" x2="477.52" y2="251.46" width="0.1524" layer="91"/>
-</segment>
-</net>
+<pinref part="PR5" gate="G$1" pin="1"/>
+</segment>
+</net>
