File: Schematics/Audio_Eagle/Filter_Stage.sch (EAGLE design)
At the start: 230 parts, among them IC1 NE5532N, IC10 NE5532N, IC11 NE5532N, IC12 NE5532N, IC13 NE5532N, IC2 NE5532N, IC3 NE5532N, IC4 NE5532N, IC5 NE5532N, IC6 NE5532N, IC7 NE5532N, P1 18AWG, U1 LME49830, U2 LME49830, U8 LME49830

Commit message: Updated Schematic
Parts:
- removed B_R_B, B_R_B1, B_R_B2, B_R_C, B_R_C1, B_R_C2, B_R_E, B_R_E1, B_R_E2: SMT_PAD_3MM, Amplifier_Parts:SMT_PAD_3MM
- removed C15: (no value), rcl:C-EU025-024X044
- removed C16, C22, C23, C27, C44, C46, C57, C58, C62, C65, C66, C72, C73, C77: 100uF, rcl:CPOL-USE2.5-6
- removed C17, C18, C24, C25, C26, C40, C42, C48, C50, C59, C60, C61, C63, C64, C67, C68, C74, C75, C76, C78, C79: 0.1uF, rcl:C-EU025-024X044
- removed C19, C20, C21, C52, C54, C56, C69, C70, C71: 22pF, rcl:C-EU025-024X044
- removed N_B, N_B1, N_B2, N_D, N_D1, N_D2, N_S, N_S1, N_S2, P_B, P_B1, P_B2, P_D, P_D1, P_D2, P_S, P_S1, P_S2: SMT_PAD_5MM, Amplifier_Parts:SMT_PAD_5MM
- removed P1: 18AWG, AWG Holes:18AWG
- removed PR1, PR2, PR3, PR4, PR5, PR6: (no value), Power Resistors:SQM
- removed R43, R57, R58, R72, R73, R87: (no value), pot:TRIM_EU-B25U
- removed R44, R47, R48, R52, R53, R54, R55, R56, R59, R62, R63, R67, R68, R69, R70, R71, R74, R77, R78, R82, R83, R84, R85, R86: 1.2k, rcl:R-US_0204/2V
- removed R45, R60, R75: 500, rcl:R-US_0204/2V
- removed R46, R61, R76: 12k, rcl:R-US_0204/2V
- removed R51, R66, R81: 10, rcl:R-US_0204/2V
- removed U$10, U$11, U$12, U$15, U$2, U$3, U$4, U$5, U$6, U$7, U$8, U$9: INDUCTOR, Amplifier_Parts:INDUCTOR
- removed U$17, U$22: MOLEX_6P, Amplifier_Parts:MOLEX_6P
- removed U1, U2, U8: LME49830, texas:LME49830
- added J1, J2, J3: MOLEX_RT_3PIN_MINIFIT, Amplifier_Parts:MOLEX_RT_3PIN_MINIFIT
- added L1, L10: 3.3mH, rcl:L-US6000-XXX-RC
- added L11, L12, L2, L3: 38mH, rcl:L-US6000-XXX-RC
- added L4, L5, L8, L9: 1.5mH, rcl:L-US6000-XXX-RC
- added L6, L7: 80mH, rcl:L-US6000-XXX-RC
- C1, C10: value (none) -> 7.4uF
- C11, C12, C3: value (none) -> 660nF
- C2: value 100uF -> 660nF; device rcl:CPOL-USE2.5-6 -> rcl:C-EU025-024X044
- C4, C9: value (none) -> 320nF
- C5, C6, C7, C8: value (none) -> 16uF
- R1, R2: value (none) -> 10k
- R10, R14, R15, R22, R23, R27, R28, R3, R31, R32, R4, R9: value (none) -> 50
- R12, R13, R17, R20, R21, R25, R26, R36, R38, R5, R7, R8: value (none) -> 1k
- R18, R29, R30, R34, R35, R37: value (none) -> 2k
- R39, R40, R41, R88, R89, R90, R91, R92: value (none) -> 100
- U$1, U$13, U$14, U$19, U$20, U$21: value TONE_POT_2GANG -> 10k
- U$16, U$18: value VOL_POT_2GANG -> 10k
Connections:
- net N$54 renamed MVO
- removed net N$100: C78.2, R83.1, R84.1, U2.IN+
- removed net N$101: C79.2, R85.2
- removed net N$102: R85.1, R87.A, U2.IN-
- removed net N$103: R86.2, R87.E, R87.S
- removed net N$105: U$22.S1
- removed net N$106: N_S1.PAD, PR3.1
- removed net N$109: N_S2.PAD, PR2.1
- removed net N$110: N_S.PAD, PR5.1
- removed net N$113: R69.2, R90.1
- removed net N$20: B_R_B1.PAD, C54.1, R58.A, R58.S, R60.2
- removed net N$28: C52.2, R59.2, U1.BIAS_P
- removed net N$31: R55.1, R57.A, U8.IN-
- removed net N$36: C42.2, R55.2
- removed net N$39: B_R_E1.PAD, C52.1, C56.1, R60.1, U1.BIAS_M
- removed net N$4 (its old number): R48.2, U8.N_OUT
- removed net N$40: R56.2, R57.E, R57.S
- removed net N$48: C56.2, U1.COMP
- removed net N$51: R62.2, U1.P_OUT
- removed net N$52: P_B1.PAD, R61.2, R63.1
- removed net N$62: N_B1.PAD, R61.1, R62.1
- removed net N$65: B_R_C.PAD, C20.2, R43.E, R44.1
- removed net N$66: C21.2, U8.COMP
- removed net N$67: B_R_E.PAD, C19.1, C21.1, R45.1, U8.BIAS_M
- removed net N$68: B_R_B.PAD, C20.1, R43.A, R43.S, R45.2
- removed net N$69: C19.2, R44.2, U8.BIAS_P
- removed net N$70: R47.2, U8.P_OUT
- removed net N$71: PR4.2, P_S1.PAD
- removed net N$72: P_B.PAD, R46.2, R48.1
- removed net N$73: N_B.PAD, R46.1, R47.1
- removed net N$74: PR6.2, P_S.PAD
- removed net N$75: PR5.2, PR6.1, R51.2, R56.1, U$17.S, U8.OSENSE
- removed net N$76: PR3.2, PR4.1, R66.2, R71.1, U$17.S2, U1.OSENSE
- removed net N$77: C61.2, R66.1
- removed net N$78: C62.+, R67.2, U1.MUTE
- removed net N$79: R63.2, U1.N_OUT
- removed net N$8 (its old number): B_R_C1.PAD, C54.2, R58.E, R59.1
- removed net N$80: C63.2, R68.1, R69.1, U1.IN+
- removed net N$81: C64.2, R70.2
- removed net N$82: R70.1, R72.A, U1.IN-
- removed net N$83: R71.2, R72.E, R72.S
- removed net N$84: C26.2, R51.1
- removed net N$85: C27.+, R52.2, U8.MUTE
- removed net N$86: B_R_C2.PAD, C70.2, R73.E, R74.1
- removed net N$87: B_R_B2.PAD, C70.1, R73.A, R73.S, R75.2
- removed net N$89: C69.2, R74.2, U2.BIAS_P
- removed net N$90: B_R_E2.PAD, C69.1, C71.1, R75.1, U2.BIAS_M
- removed net N$91: C71.2, U2.COMP
- removed net N$92: R77.2, U2.P_OUT
- removed net N$93: P_B2.PAD, R76.2, R78.1
- removed net N$94: N_B2.PAD, R76.1, R77.1
- removed net N$95: PR1.2, P_S2.PAD
- removed net N$96: PR1.1, PR2.2, R81.2, R86.1, U$17.S4, U2.OSENSE
- removed net N$97: C76.2, R81.1
- removed net N$98: C77.+, R82.2, U2.MUTE
- removed net N$99: R78.2, U2.N_OUT
- removed net V+: C16.+, C18.1, C46.+, C50.1, C66.+, C68.1, U1.+VCC, U2.+VCC, U8.+VCC
- removed net V-: C17.2, C2.-, C23.-, C25.2, C44.-, C48.2, C58.-, C60.2, C65.-, C67.2, C73.-, C75.2, N_D.PAD, N_D1.PAD, N_D2.PAD, U1.-VEE, U2.-VEE, U8.-VEE
- removed net VCC: C22.+, C24.1, C57.+, C59.1, C72.+, C74.1, P_D.PAD, P_D1.PAD, P_D2.PAD
- new net N$19: J3.2, R41.2, R90.1
- net +12V: now also J2.1; no longer U$22.S
- net -12V: now also J2.2; no longer U$22.S5
- net GND: now also C11.2, C12.2, C2.2, C3.2, C5.2, C6.2, J1.3, J2.3, L11.2, L12.1, L2.1, L3.2, L4.2, L5.2, L8.1, L9.2; no longer C10.1, C11.1, C14.2, C15.2, C16.-, C17.1, C18.2, C2.+, C22.-, C23.+, C24.2, C25.1, C26.1, C27.-, C3.1, C4.1, C40.1, C42.1, C44.+, C46.-, C48.1, C50.2, C57.-, C58.+, C59.2, C60.1, C61.1, C62.-, C63.1, C64.1, C65.+, C66.-, C67.1, C68.2, C72.-, C73.+, C74.2, C75.1, C76.1, C77.-, C78.1, C79.1, R53.2, R68.2, R83.2, U$10.1, U$11.1, U$12.1, U$17.S1, U$17.S3, U$17.S5, U$22.S3, U$3.1, U$4.1, U$5.1, U$6.1, U$9.1, U1.GND, U2.GND, U8.GND
- net N$10: no longer R54.2
- net N$104: now also C1.2, C3.1, L3.1; no longer C6.2, C8.1, U$5.2
- net N$108: now also J1.2; no longer U$22.S4
- net N$12: now also C5.1, L6.1; no longer C3.2, U$2.2
- net N$13: now also C4.2, L5.1; no longer C5.2, U$3.2
- net N$14: now also C8.1, L7.2; no longer C11.2, U$8.1
- net N$16: now also J3.1; no longer C40.2, R53.1, R54.1, U8.IN+
- net N$2: now also C13.1; no longer C1.1
- net N$22: now also C13.2; no longer C1.2
- net N$23: now also C2.1, L1.1, L2.2; no longer C7.1, U$6.2, U$7.2
- net N$26: now also J1.1; no longer U$22.S2
- net N$29: now also C1.1, L1.2; no longer C6.1, U$7.1
- net N$30: now also C9.2, L8.2; no longer C12.2, U$9.2
- net N$34: now also C11.1, L10.1, L12.2; no longer C14.1, U$12.2, U$15.2
- net N$35: now also C10.1, L10.2; no longer C13.1, U$15.1
- net N$38: now also J3.3; no longer R84.2
- net N$44: now also C7.1, L7.1; no longer C10.2, U$8.2
- net N$5: now also C14.1; no longer C9.1
- net N$59: now also C10.2, C12.1, L11.1; no longer C13.2, C15.1, U$11.2
- net N$60: now also C14.2; no longer C9.2
- net N$61: now also C9.1, L9.1; no longer C12.1, U$10.2
- net N$63: now also C4.1, L4.1; no longer C5.1, U$4.2
- net N$7: now also C6.1, L6.2; no longer C4.2, U$2.1
Other:
- note added: "Bass"
- note removed: "Bass Amp"
- note removed: "Left Amp"
- note removed: "MOSFET_n"
- note removed: "MOSFET_p"
- note removed: "Mute"
- note removed: "Right Amp"
- note removed: "Vbe multiplier"
- note removed: "altleast .5W"
- note removed: "change footprint"
- moved on the sheet: C1, C10, C11, C12, C13, C14, C29, C3, C31, C33, C35, C36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
