File: Schematics/filters/filters_V1.1.brd (EAGLE design)
At the start: 101 x 47.9 mm, 111 parts, among them IC1 NE5532N, IC2 NE5532N, IC3 NE5532N, IC4 NE5532N, IC5 NE5532N, IC6 NE5532N, IC7 NE5532N, J1 3_PIN_AMPCONN, J2 3_PIN_AMPCONN, J3 3_PIN_AMPCONN

Commit message: final board update before order
Parts:
- J2: value 3_PIN_AMPCONN -> 4_PIN_AMPCONN; device Amplifier_Parts:3_PIN_AMPCONN -> Amplifier_Parts:4_PIN_AMPCON
- moved C6 14.6 mm to (71.1, 42.5)
- moved C8 9.21 mm to (87.3, 42.5), turned to 180 degrees
- moved U$1 8.63 mm to (2.86, 9.84), turned to 90 degrees
- moved L7 1.91 mm to (95.2, 42.2)
- moved L6 1.27 mm to (87.0, 36.5)
- moved L9 0.95 mm to (79.1, 42.2)
- moved J2 0.71 mm to (97.5, 21.3)
Connections:
- net GND: now also J2.4, VR2.P$3, VR2.P$4, VR3.P$3, VR3.P$4, VR4.P$3, VR4.P$4
Routing:
- net N$7: track 33.5 -> 45.0 mm
- net N$14: track 27.6 -> 36.0 mm
- net N$19: track 29.1 -> 31.0 mm
- net N$38: track 90.5 -> 92.4 mm
- net N$10: track 76.8 -> 78.4 mm
- net N$12: track 73.2 -> 74.5 mm
- net N$61: track 32.5 -> 33.0 mm
- net N$44: track 108.3 -> 107.8 mm
Other:
- board text added: "Audio HP,BP,LP Filters"
- board text added: "Sept, 2015"
