File: Schematics/filters/filters_V1.1.Carlos.sch (EAGLE design)
At the start: 107 parts, among them J1 4_PIN_AMPCONN, J10 OSTVN03A150, J11 OSTVN03A150, J12 OSTVN03A150, J13 OSTVN03A150, J14 OSTVN03A150, J2 1984633, J3 2TERMINAL_SPEAKER, J4 2TERMINAL_SPEAKER, J5 2TERMINAL_SPEAKER, J6 OSTVN03A150, J7 OSTVN03A150, J8 OSTVN03A150, J9 OSTVN03A150, U1 LME49830, U2 LME49830, U3 LME49830

Commit message: added coloring diagram for transistors
Parts:
- removed C15, C18, C19, C25, C26, C27, C34, C40, C42: 0.1uF, rcl:C-EU050-024X044
- removed C16, C17, C23, C24, C28, C32: 100uF, rcl:CPOL-USE2.5-6
- removed C20, C21, C22, C44: 22pF, rcl:C-EU050-024X044
- removed C30: 200uF, rcl:C-EU050-024X044
- removed J10, J11, J12, J13, J14, J6, J7, J8, J9: OSTVN03A150, Amplifier_Parts:OSTVN03A150
- removed J4, J5: 2TERMINAL_SPEAKER, Amplifier_Parts:2TERMINAL_SPEAKER
- removed PR1, PR2, PR3, PR4, PR5, PR6: 0.1, rcl:R-US_0617/5V
- removed R51: 10, rcl:R-US_0309/V
- removed R52: 4.7k, rcl:R-US_0204/2V
- removed R55: 240, rcl:R-US_0204/2V
- removed R56: 6.8k, rcl:R-US_0204/2V
- removed U1, U2, U3: LME49830, LME49830_1:LME49830
- removed VR5: 20k, Amplifier_Parts:EVM2W
- removed VR6: 10k, Amplifier_Parts:EVM2W
- added C47, C49, C51, C53, C55: 0.1uF, rcl:C-US050-024X044
- added IC1, IC2, IC3, IC4, IC5, IC6, IC7: NE5532N, linear:NE5532N
- added L1, L10: 3.3mH, rcl:L-US6000-XXX-RC
- added L11, L12, L2, L3: 38mH, rcl:L-US6000-XXX-RC
- added L4, L5, L8, L9: 1.5mH, rcl:L-US6000-XXX-RC
- added L6, L7: 80mH, rcl:L-US6000-XXX-RC
- added R25, R36: 3.3k, rcl:R-US_0204/2V
- added R26, R38: 1k, rcl:R-US_0204/2V
- added R27, R28, R31, R32: 50, rcl:R-US_0204/2V
- added R29, R30, R34, R35, R37: 2.7k, rcl:R-US_0204/2V
- added R33: 12k, rcl:R-US_0204/2V
- added R39, R40, R41, R88, R89, R90, R91, R92: 100, rcl:R-US_0204/2V
- added R42, R43, R49: 4.7k, rcl:R-US_0204/2V
- C1, C10: value 22pF -> 7.4uF; device rcl:C-EU050-024X044 -> rcl:C-US050-024X044
- C11, C3: value 0.1uF -> 660nF; device rcl:C-EU050-024X044 -> rcl:C-US050-024X044
- C12, C2: value 100uF -> 660nF; device rcl:CPOL-USE2.5-6 -> rcl:C-US050-024X044
- C13: value 0.1uF -> 100u; device rcl:C-EU050-024X044 -> rcl:C-US050-024X044
- C14: value 100uF -> 100u; device rcl:CPOL-USE2.5-6 -> rcl:C-US050-024X044
- C29, C35, C37: value 22pF -> 0.1uF; device rcl:C-EU050-024X044 -> rcl:C-US050-024X044
- C31, C39, C43: value 100uF -> 0.1uF; device rcl:CPOL-USE2.5-6 -> rcl:C-US050-024X044
- C33, C41, C45: device rcl:C-EU050-024X044 -> rcl:C-US050-024X044
- C36: value 22pF -> 100uF; device rcl:C-EU050-024X044 -> rcl:CPOL-USE2.5-6
- C4: value 100uF -> 320nF; device rcl:CPOL-USE2.5-6 -> rcl:C-US050-024X044
- C5: value 0.1uF -> 16uF; device rcl:C-EU050-024X044 -> rcl:C-US050-024X044
- C6: value 100uF -> 16uF; device rcl:CPOL-USE2.5-6 -> rcl:C-US050-024X044
- C7: value 200uF -> 16uF; device rcl:C-EU050-024X044 -> rcl:C-US050-024X044
- C8: value 22pF -> 16uF; device rcl:C-EU050-024X044 -> rcl:C-US050-024X044
- C9: value 22pF -> 320nF; device rcl:C-EU050-024X044 -> rcl:C-US050-024X044
- J1: value 4_PIN_AMPCONN -> 3_PIN_AMPCONN; device Amplifier_Parts:4_PIN_AMPCONN -> Amplifier_Parts:3_PIN_AMPCONN
- J2: value 1984633 -> 4_PIN_AMPCONN; device Amplifier_Parts:1984633 -> Amplifier_Parts:4_PIN_AMPCONN
- J3: value 2TERMINAL_SPEAKER -> 3_PIN_AMPCONN; device Amplifier_Parts:2TERMINAL_SPEAKER -> Amplifier_Parts:3_PIN_AMPCONN
- R1: value 240 -> 8.2k
- R10: value 6.8k -> 50
- R11: value 240 -> 12k
- R12: value 240 -> 3.3k
- R13: value 6.8k -> 1k
- R14, R3: value 1.2k -> 50
- R15, R4: value 500 -> 50
- R17: value 120 -> 3.3k
- R18: value 120 -> 2.7k
- R19: value 10 -> 12k; device rcl:R-US_0309/V -> rcl:R-US_0204/2V
- R2: value 6.8k -> 8.2k
- R20: value 4.7k -> 1k
- R21: value 6.8k -> 3.3k
- R22, R23: value 240 -> 50
- R24: value 6.8k -> 12k
- R44: value 1.2k -> 4.7k
- R45: value 500 -> 4.7k
- R46: value 12k -> 4.7k
- R47, R48: value 120 -> 4.7k
- R5: value 12k -> 1k
- R6: value 120 -> 12k
- R7: value 120 -> 1k
- R8: value 10 -> 5.6k; device rcl:R-US_0309/V -> rcl:R-US_0204/2V
- R9: value 4.7k -> 50
- VR1: value 20k -> 10k; device Amplifier_Parts:EVM2W -> Amplifier_Parts:VOL_POT_2GANG
- VR2, VR4: device Amplifier_Parts:EVM2W -> Amplifier_Parts:P140KV1-F25BR
- VR3: value 20k -> 10k; device Amplifier_Parts:EVM2W -> Amplifier_Parts:P140KV1-F25BR
Connections:
- removed net BASS_IN: J1.2, R11.2
- removed net BASS_OUT: J4.1, PR1.2, PR2.1, R13.1, R8.2, U2.ONSENSE
- removed net B_NMOS_G: J10.2, R5.2, R7.1
- removed net B_NMOS_S: J10.3, PR2.2
- removed net B_PMOS_G: J9.2, R5.1, R6.1
- removed net B_PMOS_S: J9.1, PR1.1
- removed net B_VBE_B: C21.1, J11.2, R4.2, VR4.A, VR4.B
- removed net B_VBE_C: C21.2, J11.3, R3.1, VR4.C
- removed net B_VBE_E: C20.1, C22.1, J11.1, R4.1, U2.BIASM
- removed net LEFT_OUT: J5.1, PR3.2, PR4.1, R19.2, R24.1, U3.ONSENSE
- removed net L_NMOS_G: J12.2, R16.2, R18.1
- removed net L_NMOS_S: J12.3, PR4.2
- removed net L_PMOS_G: J13.2, R16.1, R17.1
- removed net L_PMOS_S: J13.1, PR3.1
- removed net L_VBE_B: C36.1, J14.2, R15.2, VR6.A, VR6.B
- removed net L_VBE_C: C36.2, J14.3, R14.1, VR6.C
- removed net L_VBE_E: C35.1, C37.1, J14.1, R15.1, U3.BIASM
- removed net MUTE: J2.2, R20.1, R52.1, R9.1
- removed net N$19: R12.1, U2.IN-, VR3.A
- removed net N$38: R18.2, U3.NOUT
- removed net N$66: C8.2, U1.COMP
- removed net N$69: C9.2, R44.2, U1.BIASP
- removed net N$70: R47.2, U1.POUT
- removed net N$84: C15.2, R51.1
- removed net N$85: C6.+, R52.2, U1.MUTE
- removed net RIGHT_OUT: J3.1, PR5.2, PR6.1, R51.2, R56.1, U1.ONSENSE
- removed net R_NMOS_G: J6.2, R46.2, R48.1
- removed net R_NMOS_S: J6.3, PR6.2
- removed net R_PMOS_G: J8.2, R46.1, R47.1
- removed net R_PMOS_S: J8.1, PR5.1
- removed net R_VBE_B: C10.1, J7.2, R45.2, VR2.A, VR2.B
- removed net R_VBE_C: C10.2, J7.3, R44.1, VR2.C
- removed net R_VBE_E: C8.1, C9.1, J7.1, R45.1, U1.BIASM
- removed net V+: C11.1, C12.+, C17.+, C19.1, C23.+, C25.1, C32.+, C34.1, C38.+, C4.+, C40.1, C5.1, J10.1, J12.1, J2.4, J6.1, U1.+VCC, U2.+VCC, U3.+VCC
- removed net V-: C13.2, C14.-, C16.-, C18.2, C2.-, C24.-, C26.2, C3.2, C31.-, C33.2, C39.-, C41.2, J13.3, J2.3, J8.3, J9.3, U1.-VEE, U2.-VEE, U3.-VEE
- new net +12V: C31.2, C35.2, C36.+, C39.2, C43.2, C47.2, C51.2, C55.2, IC1P.V+, IC2P.V+, IC3P.V+, IC4P.V+, IC5P.V+, IC6P.V+, IC7P.V+, J3.2
- new net -12V: C29.1, C33.1, C37.1, C38.-, C41.1, C45.1, C49.1, C53.1, IC1P.V-, IC2P.V-, IC3P.V-, IC4P.V-, IC5P.V-, IC6P.V-, IC7P.V-, J3.1
- new net BASS: J2.2, R41.2, R90.2
- new net LEFT: J2.3, R39.2, R91.2, R92.2
- new net MVO: IC6B.OUT, R40.1, R90.1, VR4A.1_2, VR4A.1_3
- new net N$1: IC1A.-IN, R1.2, VR1A.1
- new net N$104: C1.2, C3.1, IC2A.+IN, L3.1, R15.2
- new net N$11: IC6B.-IN, R34.1, R6.1
- new net N$12: C5.1, L6.1, R4.2
- new net N$2: C13.1, IC1A.OUT, VR1A.2, VR1A.3
- new net N$21: IC2B.OUT, R88.1, VR2A.1_2, VR2A.1_3
- new net N$22: C13.2, R14.1, R4.1, R9.1
- new net N$23: C2.1, L1.1, L2.2, R14.2
- new net N$24: R18.2, VR2A.1_1
- new net N$29: C1.1, L1.2
- new net N$30: C9.2, L8.2, R22.2
- new net N$32: IC5A.OUT, R24.2, R25.2
- new net N$33: IC5B.-IN, R24.1, R30.1
- new net N$34: C11.1, L10.1, L12.2, R27.2
- new net N$44: C7.1, L7.1, R32.2
- new net N$45: IC7A.-IN, R20.2, R21.1
- new net N$46: IC5A.-IN, R25.1, R26.2
- new net N$47: IC3A.OUT, R33.2, R36.2
- new net N$48: IC3B.+IN, R49.2
- new net N$49: IC7B.+IN, R47.2
- new net N$5: C14.1, IC1B.OUT, VR1B.2, VR1B.3
- new net N$50: IC3B.OUT, R92.1, VR2B.1_2, VR2B.1_3
- new net N$53: R34.2, VR4A.1_1
- new net N$55: IC4B.OUT, R89.1, VR3A.1_2, VR3A.1_3
- new net N$56: R35.2, VR3A.1_1
- new net N$57: R37.2, VR2B.1_1
- new net N$58: IC3A.-IN, R36.1, R38.2
- new net N$59: C10.2, C12.1, IC3A.+IN, L11.1, R28.2
- new net N$60: C14.2, R22.1, R27.1, R32.1
- new net N$61: C9.1, IC5A.+IN, L9.1, R23.2
- new net N$63: C4.1, IC4A.+IN, L4.1, R10.2
- new net N$8: IC3B.-IN, R33.1, R37.1
- new net N$88: IC6A.OUT, R6.2, R8.2
- new net N$9: IC4A.-IN, R12.1, R13.2
- new net RIGHT: J2.1, R40.2, R88.2, R89.2
- net GND: now also C12.2, C2.2, C29.2, C3.2, C31.1, C33.2, C35.1, C36.-, C37.2, C38.+, C39.1, C41.2, C43.1, C45.2, C47.1, C49.2, C51.1, C53.2, C55.1, C6.2, C7.2, C8.2, J1.3, J2.4, J3.3, L11.2, L12.1, L2.1, L3.2, L4.2, L5.2, L8.1, L9.2, R10.1, R13.1, R15.1, R20.1, R23.1, R26.1, R28.1, R3.1, R31.1, R38.1, R42.1, R43.1, R44.2, R45.1, R46.1, R47.1, R48.1, R49.1, R5.1, R7.1, VR2G$1.TAB, VR2G$2.TAB, VR3G$1.TAB, VR3G$2.TAB, VR4G$1.TAB, VR4G$2.TAB; no longer C1.1, C12.-, C13.1, C14.+, C15.1, C16.+, C17.-, C18.1, C19.2, C2.+, C23.-, C24.+, C25.2, C26.1, C27.1, C28.-, C29.1, C3.1, C30.1, C31.+, C32.-, C33.1, C34.2, C38.-, C39.+, C4.-, C40.2, C41.1, C42.1, C43.-, C44.1, C45.1, C6.-, C7.1, J1.4, J2.1, J3.2, J4.2, J5.2, R10.2, R2.2, R21.2, U1.GND, U2.GND, U3.GND
- net LEFT_IN: now also J1.2, R2.1; no longer J1.3, R22.2
- net N$13: now also C4.2, L5.1, R9.2; no longer C27.2, R8.1
- net N$14: now also C8.1, IC7A.+IN, L7.2, R31.2; no longer C28.+, R9.2, U2.MUTE
- net N$15: now also IC2A.OUT, R16.2, R17.2; no longer R7.2, U2.NOUT
- net N$16: now also IC1A.+IN, R42.2; no longer C1.2, R1.1, R2.1, U1.IN+
- net N$17: now also IC4A.OUT, R11.2, R12.2; no longer C29.2, R10.1, R11.1, U2.IN+
- net N$18: now also IC4B.-IN, R11.1, R35.1; no longer C30.2, R12.2
- net N$20: now also IC1B.+IN, R43.2; no longer R13.2, VR3.B, VR3.C
- net N$25: now also IC7B.-IN, R19.1, R29.1; no longer C35.2, R14.2, U3.BIASP
- net N$27: now also IC2A.-IN, R17.1, R5.2; no longer C37.2, U3.COMP
- net N$28: now also IC2B.+IN, R44.1; no longer R17.2, U3.POUT
- net N$3: now also IC1B.-IN, R2.2, VR1B.1; no longer C20.2, R3.2, U2.BIASP
- net N$31: now also IC5B.+IN, R48.2; no longer R55.1, U1.IN-, VR1.A
- net N$35: now also C10.1, L10.2; no longer C42.2, R19.1
- net N$36: now also IC4B.+IN, R45.2; no longer C7.2, R55.2
- net N$37: now also R29.2, VR4B.1_1; no longer C43.+, R20.2, U3.MUTE
- net N$39: now also IC6B.+IN, R46.2; no longer C44.2, R21.1, R22.1, U3.IN+
- net N$4: now also IC2B.-IN, R16.1, R18.1; no longer R48.2, U1.NOUT
- net N$40: now also IC7B.OUT, R39.1, R41.1, VR4B.1_2, VR4B.1_3; no longer R56.2, VR1.B, VR1.C
- net N$41: now also IC5B.OUT, R91.1, VR3B.1_2, VR3B.1_3; no longer C45.2, R23.2
- net N$42: now also R30.2, VR3B.1_1; no longer R23.1, U3.IN-, VR5.A
- net N$43: now also IC7A.OUT, R19.2, R21.2; no longer R24.2, VR5.B, VR5.C
- net N$6: now also IC6A.-IN, R7.2, R8.1; no longer C22.2, U2.COMP
- net N$7: now also C6.1, IC6A.+IN, L6.2, R3.2; no longer R6.2, U2.POUT
- net RIGHT_IN: now also R1.1; no longer R1.2
Other:
- note added: "BASS LEFT CHANNEL"
- note added: "BASS RIGHT CHANNEL"
- note added: "Bass"
- note added: "Left"
- note added: "MIDS LEFT CHANNEL"
- note added: "MIDS RIGHT CHANNEL"
- note added: "Right"
- note added: "TREBLE LEFT CHANNEL"
- note added: "TREBLE RIGHT CHANNEL"
- note added: "cut this resisiotr to remove 2 bass"
- note added: "short this resistor to have bass on left channel"
- note removed: "250V"
- note removed: "B_PMOS_D"
- note removed: "Bass Amp"
- note removed: "L_NMOS_D"
- note removed: "L_PMOS_D"
- note removed: "Left Amp"
- note removed: "MOSFET_n"
- note removed: "MOSFET_p"
- note removed: "R_NMOS_D"
- note removed: "R_PMOS_D"
- note removed: "Right Amp"
- note removed: "Vbe multiplier"
- note removed: "altleast 2W"
- note removed: "change footprint"
- moved on the sheet: C1, C10, C11, C13, C29, C3, C33, C35, C37, C38, C41, C45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
