File: Schematics/PA/Power_Amp_V1.0.brd (EAGLE design)
At the start: 83.5 x 71.1 mm, 123 parts, among them J1 4_PIN_AMPCONN, U1 LME49830, U2 LME49830, U3 LME49830, X1 5566-4

Commit message: added part values to PA from breadboard prototype
Parts:
- C22: value 22pF -> 20pF
- C29: value 0.1uF -> 22pF
- C30: value 0.1uF -> 200uF
- R10, R13: value 1.2k -> 6.8k
- R11, R12: value 1.2k -> 270
- R20, R52, R9: value 1.2k -> 4.7k
- R4: value 500 -> 470
Changed lines of the file:
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@@
 <?xml version="1.0" encoding="utf-8"?>
 <!DOCTYPE eagle SYSTEM "eagle.dtd">
-<eagle version="7.4.0">
+<eagle version="6.5.0">
 <drawing>
 <settings>
@@
 <pass name="Default">
 <param name="RoutingGrid" value="50mil"/>
-<param name="AutoGrid" value="1"/>
-<param name="Efforts" value="0"/>
-<param name="TopRouterVariant" value="1"/>
 <param name="tpViaShape" value="round"/>
-<param name="PrefDir.1" value="a"/>
+<param name="PrefDir.1" value="|"/>
 <param name="PrefDir.2" value="0"/>
 <param name="PrefDir.3" value="0"/>
@@
 <param name="PrefDir.14" value="0"/>
 <param name="PrefDir.15" value="0"/>
-<param name="PrefDir.16" value="a"/>
+<param name="PrefDir.16" value="-"/>
 <param name="cfVia" value="8"/>
 <param name="cfNonPref" value="5"/>
@@
 <element name="C20" library="rcl" package="C050-024X044" value="22pF" x="36.83" y="39.37"/>
 <element name="C21" library="rcl" package="C050-024X044" value="22pF" x="54.61" y="45.72"/>
-<element name="C22" library="rcl" package="C050-024X044" value="22pF" x="40.64" y="31.75"/>
+<element name="C22" library="rcl" package="C050-024X044" value="20pF" x="40.64" y="31.75"/>
 <element name="C23" library="rcl" package="E2,5-6" value="100uF" x="21.59" y="10.16" rot="R270"/>
 <element name="C24" library="rcl" package="E2,5-6" value="100uF" x="16.51" y="10.16" rot="R270"/>
@@
 <element name="C27" library="rcl" package="C050-024X044" value="0.1uF" x="31.75" y="33.02"/>
 <element name="C28" library="rcl" package="E2,5-6" value="100uF" x="21.59" y="27.94" rot="R270"/>
-<element name="C29" library="rcl" package="C050-024X044" value="0.1uF" x="15.24" y="36.83"/>
+<element name="C29" library="rcl" package="C050-024X044" value="22pF" x="15.24" y="36.83"/>
 <element name="C3" library="rcl" package="C050-024X044" value="0.1uF" x="30.48" y="59.69"/>
-<element name="C30" library="rcl" package="C050-024X044" value="0.1uF" x="15.24" y="43.18"/>
+<element name="C30" library="rcl" package="C050-024X044" value="200uF" x="15.24" y="43.18"/>
 <element name="C31" library="rcl" package="E2,5-6" value="100uF" x="11.43" y="10.16" rot="R270"/>
 <element name="C32" library="rcl" package="E2,5-6" value="100uF" x="36.83" y="27.94" rot="R270"/>
@@
 <element name="P_S_3" library="Amplifier_Parts" package="18AWG_HOLE" value="" x="13.97" y="2.54"/>
 <element name="R1" library="rcl" package="0204V" value="1.2k" x="37.7825" y="52.3875" rot="R180"/>
-<element name="R10" library="rcl" package="0204V" value="1.2k" x="36.83" y="34.29"/>
-<element name="R11" library="rcl" package="0204V" value="1.2k" x="17.78" y="39.37"/>
-<element name="R12" library="rcl" package="0204V" value="1.2k" x="54.61" y="38.1"/>
-<element name="R13" library="rcl" package="0204V" value="1.2k" x="31.75" y="38.1"/>
+<element name="R10" library="rcl" package="0204V" value="6.8k" x="36.83" y="34.29"/>
+<element name="R11" library="rcl" package="0204V" value="270" x="17.78" y="39.37"/>
+<element name="R12" library="rcl" package="0204V" value="270" x="54.61" y="38.1"/>
+<element name="R13" library="rcl" package="0204V" value="6.8k" x="31.75" y="38.1"/>
 <element name="R14" library="rcl" package="0204V" value="1.2k" x="8.89" y="19.05"/>
 <element name="R15" library="rcl" package="0204V" value="500" x="21.59" y="17.78"/>
@@
 <element name="R19" library="rcl" package="0309V" value="10" x="62.23" y="12.7"/>
 <element name="R2" library="rcl" package="0204V" value="1.2k" x="41.275" y="51.1175" rot="R270"/>
-<element name="R20" library="rcl" package="0204V" value="1.2k" x="31.75" y="15.24"/>
+<element name="R20" library="rcl" package="0204V" value="4.7k" x="31.75" y="15.24"/>
 <element name="R21" library="rcl" package="0204V" value="1.2k" x="35.56" y="6.35"/>
 <element name="R22" library="rcl" package="0204V" value="1.2k" x="38.1" y="10.16"/>
@@
 <element name="R24" library="rcl" package="0204V" value="1.2k" x="58.42" y="16.51"/>
 <element name="R3" library="rcl" package="0204V" value="1.2k" x="26.67" y="38.1"/>
-<element name="R4" library="rcl" package="0204V" value="500" x="31.75" y="35.56"/>
+<element name="R4" library="rcl" package="0204V" value="470" x="31.75" y="35.56"/>
 <element name="R44" library="rcl" package="0204V" value="1.2k" x="34.29" y="73.66"/>
 <element name="R45" library="rcl" package="0204V" value="500" x="11.43" y="66.04"/>
@@
 <element name="R5" library="rcl" package="0204V" value="12k" x="34.29" y="41.91"/>
 <element name="R51" library="rcl" package="0309V" value="10" x="68.58" y="66.675" rot="R270"/>
-<element name="R52" library="rcl" package="0204V" value="1.2k" x="22.86" y="67.31"/>
+<element name="R52" library="rcl" package="0204V" value="4.7k" x="22.86" y="67.31"/>
 <element name="R55" library="rcl" package="0204V" value="1.2k" x="40.3225" y="54.61" rot="R180"/>
 <element name="R56" library="rcl" package="0204V" value="1.2k" x="64.77" y="65.405" rot="R180"/>
@@
 <element name="R7" library="rcl" package="0204V" value="1.2k" x="40.64" y="40.64"/>
 <element name="R8" library="rcl" package="0309V" value="10" x="57.15" y="33.02"/>
-<element name="R9" library="rcl" package="0204V" value="1.2k" x="16.51" y="34.29"/>
+<element name="R9" library="rcl" package="0204V" value="4.7k" x="16.51" y="34.29"/>
 <element name="U$17" library="Amplifier_Parts" package="MOLEX_6P" value="MOLEX_6P" x="82.55" y="35.56" rot="R90"/>
 <element name="VR1" library="Amplifier_Parts" package="EVM2W" value="" x="61.2775" y="64.4525"/>
