File: Schematics/PA/Power_Amp_V1.0.sch (EAGLE design)
At the start: 228 parts, among them IC1 NE5532N, IC10 NE5532N, IC11 NE5532N, IC12 NE5532N, IC13 NE5532N, IC2 NE5532N, IC3 NE5532N, IC4 NE5532N, IC5 NE5532N, IC6 NE5532N, IC7 NE5532N, P1 18AWG, U1 LME49830, U2 LME49830, U8 LME49830

Commit message: began work on the Power Amp
Parts:
- removed C46, C57, C58, C62, C65, C66, C72, C73, C77: 100uF, rcl:CPOL-USE2.5-6
- removed C47, C48, C49, C50, C51, C53, C55, C59, C60, C61, C63, C64, C67, C68, C74, C75, C76, C78, C79: 0.1uF, rcl:C-EU025-024X044
- removed C52, C54, C56, C69, C70, C71: 22pF, rcl:C-EU025-024X044
- removed IC1, IC10, IC11, IC12, IC13, IC2, IC3, IC4, IC5, IC6, IC7: NE5532N, linear:NE5532N
- removed P1: 18AWG, AWG Holes:18AWG
- removed R27, R28, R29, R30, R31, R32, R33, R34, R35, R36, R37, R38, R39, R88, R89, R90, R91, R92: (no value), rcl:R-US_0204/2V
- removed R58, R72, R73, R87: (no value), pot:TRIM_EU-B25U
- removed R59, R62, R63, R67, R68, R69, R70, R71, R74, R77, R78, R82, R83, R84, R85, R86: 1.2k, rcl:R-US_0204/2V
- removed R60, R75: 500, rcl:R-US_0204/2V
- removed R61, R76: 12k, rcl:R-US_0204/2V
- removed R66, R81: 10, rcl:R-US_0204/2V
- removed U$10, U$11, U$12, U$15, U$2, U$3, U$4, U$5, U$6, U$7, U$8, U$9: INDUCTOR, Amplifier_Parts:INDUCTOR
- removed U$13, U$14, U$19, U$20, U$21: TONE_POT_2GANG, Amplifier_Parts:TONE_POT_2GANG
- removed U$16, U$18: VOL_POT_2GANG, Amplifier_Parts:VOL_POT_2GANG
- removed U$22: MOLEX_6P, Amplifier_Parts:MOLEX_6P
- removed U8: LME49830, texas:LME49830
- added C28, C32: 0.1uF, rcl:C-EU025-024X044
- added C30: 100uF, rcl:CPOL-USE2.5-6
- added C34: 22pF, rcl:C-EU025-024X044
- added J1: 4_PIN_AMPCONN, Amplifier_Parts:4_PIN_AMPCONN
- added U4: LME49830, texas:LME49830
- C1, C10, C14, C3, C9: value (none) -> 100uF; device rcl:C-EU025-024X044 -> rcl:CPOL-USE2.5-6
- C11, C12, C13, C15, C4, C5: value (none) -> 0.1uF
- C29, C37, C43: value 0.1uF -> 100uF; device rcl:C-EU025-024X044 -> rcl:CPOL-USE2.5-6
- C33, C35: value 0.1uF -> 22pF
- C38, C44: value 100uF -> 0.1uF; device rcl:CPOL-USE2.5-6 -> rcl:C-EU025-024X044
- C6, C7, C8: value (none) -> 22pF
- R1, R13, R14, R26: device rcl:R-US_0204/2V -> pot:TRIM_EU-B25U
- R10, R11, R12, R15, R18, R19, R2, R21, R22, R23, R24, R25, R5, R6, R8, R9: value (none) -> 1.2k
- R16, R3: value (none) -> 500
- R17, R4: value (none) -> 12k
- R20, R7: value (none) -> 10
- U$1: value TONE_POT_2GANG -> SCREW_TERMINAL_4; device Amplifier_Parts:TONE_POT_2GANG -> Amplifier_Parts:SCREW_TERMINAL_4
Connections:
- removed net +12V: C31.2, C35.2, C36.+, C39.2, C43.2, C47.2, C51.2, C55.2, U$22.S
- removed net -12V: C29.1, C33.1, C37.1, C38.-, C41.1, C45.1, C49.1, C53.1, U$22.S5
- removed net N$100: C78.2, R83.1, R84.1, U2.IN+
- removed net N$101: C79.2, R85.2
- removed net N$102: R85.1, R87.A, U2.IN-
- removed net N$103: R86.2, R87.E, R87.S
- removed net N$104: C6.2, C8.1, IC3A.+IN, R15.2, U$5.2
- removed net N$105: U$22.S1
- removed net N$106: N_S1.PAD, PR3.1
- removed net N$108: R1.1, U$22.S4
- removed net N$109: N_S2.PAD, PR2.1
- removed net N$3: IC12A.-IN, R1.2, U$18G$1.1_1
- removed net N$45: IC10A.-IN, R20.2, R21.1
- removed net N$47: IC13A.OUT, R33.1, R36.2
- removed net N$48: C56.2, U1.COMP
- removed net N$49: IC13B.-IN, R33.2, R37.1
- removed net N$50: IC13B.OUT, R92.1, U$21G$1.1_2, U$21G$1.1_3
- removed net N$51: R62.2, U1.P_OUT
- removed net N$52: P_B1.PAD, R61.2, R63.1
- removed net N$53: R34.2, U$1G$1.1_1
- removed net N$54: IC1B.OUT, R90.1, U$1G$1.1_2, U$1G$1.1_3
- removed net N$55: IC2B.OUT, R89.1, U$13G$1.1_2, U$13G$1.1_3
- removed net N$56: R35.2, U$13G$1.1_1
- removed net N$57: R37.2, U$21G$1.1_1
- removed net N$58: IC13A.-IN, R36.1, R38.2
- removed net N$59: C13.2, C15.1, IC13A.+IN, R28.2, U$11.2
- removed net N$60: C9.2, R22.1, R27.1, R32.1
- removed net N$61: C12.1, IC11A.+IN, R23.2, U$10.2
- removed net N$62: N_B1.PAD, R61.1, R62.1
- removed net N$63: C5.1, IC2A.+IN, R10.2, U$4.2
- removed net N$64: IC10B.OUT, R39.2, R69.2, U$19G$1.1_2, U$19G$1.1_3
- removed net N$71: PR4.2, P_S1.PAD
- removed net N$76: PR3.2, PR4.1, R66.2, R71.1, U$17.S2, U1.OSENSE
- removed net N$77: C61.2, R66.1
- removed net N$78: C62.+, R67.2, U1.MUTE
- removed net N$79: R63.2, U1.N_OUT
- removed net N$80: C63.2, R68.1, R69.1, U1.IN+
- removed net N$81: C64.2, R70.2
- removed net N$82: R70.1, R72.A, U1.IN-
- removed net N$83: R71.2, R72.E, R72.S
- removed net N$86: B_R_C2.PAD, C70.2, R73.E, R74.1
- removed net N$87: B_R_B2.PAD, C70.1, R73.A, R73.S, R75.2
- removed net N$88: IC1A.OUT, R6.1, R8.2
- removed net N$89: C69.2, R74.2, U2.BIAS_P
- removed net N$90: B_R_E2.PAD, C69.1, C71.1, R75.1, U2.BIAS_M
- removed net N$91: C71.2, U2.COMP
- removed net N$92: R77.2, U2.P_OUT
- removed net N$93: P_B2.PAD, R76.2, R78.1
- removed net N$94: N_B2.PAD, R76.1, R77.1
- removed net N$95: PR1.2, P_S2.PAD
- removed net N$96: PR1.1, PR2.2, R81.2, R86.1, U$17.S4, U2.OSENSE
- removed net N$97: C76.2, R81.1
- removed net N$98: C77.+, R82.2, U2.MUTE
- removed net N$99: R78.2, U2.N_OUT
- removed net VCC: C22.+, C24.1, C57.+, C59.1, C72.+, C74.1, P_D.PAD, P_D1.PAD, P_D2.PAD
- new net MUTE: R52.1, U$1.S1
- new net MUTE1: R8.1
- new net MUTE2: R21.1
- net GND: now also C1.+, C10.+, C11.2, C12.1, C13.1, C14.-, C15.1, C28.1, C29.+, C3.-, C30.-, C32.2, C37.+, C38.2, C41.1, C43.-, C44.1, C45.1, C5.2, C9.-, J1.4, R22.2, R9.2, U$1.S2, U4.GND; no longer C10.1, C11.1, C14.2, C15.2, C29.2, C3.1, C33.2, C35.1, C37.2, C38.+, C41.2, C43.1, C44.+, C45.2, C46.-, C47.1, C48.1, C49.2, C50.2, C51.1, C53.2, C55.1, C57.-, C58.+, C59.2, C60.1, C61.1, C62.-, C63.1, C64.1, C65.+, C66.-, C67.1, C68.2, C7.2, C72.-, C73.+, C74.2, C75.1, C76.1, C77.-, C78.1, C79.1, C8.2, IC10B.+IN, IC11B.+IN, IC12A.+IN, IC13B.+IN, IC1B.+IN, IC1P.V+, IC1P.V-, IC2B.+IN, IC2P.V+, IC2P.V-, IC3B.+IN, IC3P.V+, IC3P.V-, IC4P.V+, IC4P.V-, IC5P.V+, IC5P.V-, IC6P.V+, IC6P.V-, IC7A.+IN, IC7P.V+, IC7P.V-, R10.1, R13.1, R15.1, R20.1, R23.1, R26.1, R28.1, R3.2, R31.2, R38.1, R5.1, R68.2, R7.1, R83.2, U$10.1, U$11.1, U$12.1, U$22.S3, U$3.1, U$4.1, U$5.1, U$6.1, U$9.1, U8.GND
- net N$1: now also B_R_C1.PAD, C7.2, R1.E, R2.1; no longer IC7A.-IN, R2.2, U$16G$1.1_1
- net N$10: now also J1.1; no longer R88.2, R89.2, R90.2
- net N$11: now also N_B1.PAD, R4.1, R5.1; no longer IC1B.-IN, R34.1, R6.2
- net N$12: now also PR2.2, P_S1.PAD; no longer C3.2, R4.2, U$2.2
- net N$13: now also PR1.2, PR2.1, R12.1, R7.2, U$17.S2, U4.OSENSE; no longer C5.2, R9.2, U$3.2
- net N$14: now also C13.2, R7.1; no longer C11.2, IC10A.+IN, R31.1, U$8.1
- net N$15: now also C14.+, R8.2, U4.MUTE; no longer IC3A.OUT, R16.1, R17.2
- net N$16: now also U1.IN+; no longer U8.IN+
- net N$17: now also R6.2, U4.N_OUT; no longer IC2A.OUT, R11.1, R12.2
- net N$18: now also C15.2, R10.1, R9.1, U4.IN+; no longer IC2B.-IN, R11.2, R35.1
- net N$19: now also C28.2, R11.2; no longer IC3B.-IN, R16.2, R18.1
- net N$2: now also B_R_B1.PAD, C7.1, R1.A, R1.S, R3.2; no longer C1.1, IC7A.OUT, U$16G$1.1_2, U$16G$1.1_3
- net N$20: now also R11.1, R13.A, U4.IN-; no longer B_R_B1.PAD, C54.1, R58.A, R58.S, R60.2
- net N$21: now also R12.2, R13.E, R13.S; no longer IC3B.OUT, R88.1, U$14G$1.1_2, U$14G$1.1_3
- net N$22: now also J1.2, R10.2; no longer C1.2, R14.1, R4.1, R9.1
- net N$23: now also N_S1.PAD, PR1.1; no longer C7.1, R14.2, U$6.2, U$7.2
- net N$24: now also B_R_C2.PAD, C34.2, R14.E, R15.1; no longer R18.2, U$14G$1.1_1
- net N$25: now also B_R_B2.PAD, C34.1, R14.A, R14.S, R16.2; no longer IC10B.-IN, R19.2, R29.1
- net N$26: now also C33.2, R15.2, U2.BIAS_P; no longer R2.1, U$22.S2
- net N$27: now also B_R_E2.PAD, C33.1, C35.1, R16.1, U2.BIAS_M; no longer IC3A.-IN, R17.1, R5.2
- net N$28: now also C35.2, U2.COMP; no longer C52.2, R59.2, U1.BIAS_P
- net N$29: now also J1.3, R23.2; no longer C6.1, U$7.1
- net N$30: now also R18.2, U2.P_OUT; no longer C12.2, R22.2, U$9.2
- net N$31: now also U1.IN-; no longer U8.IN-
- net N$32: now also P_B2.PAD, R17.2, R19.1; no longer IC11A.OUT, R24.1, R25.2
- net N$33: now also N_B2.PAD, R17.1, R18.1; no longer IC11B.-IN, R24.2, R30.1
- net N$34: now also PR4.2, P_S2.PAD; no longer C14.1, R27.2, U$12.2, U$15.2
- net N$35: now also PR3.2, PR4.1, R20.2, R25.1, U$17.S4, U2.OSENSE; no longer C13.1, U$15.1
- net N$37: now also C41.2, R20.1; no longer R29.2, U$19G$1.1_1
- net N$38: now also C43.+, R21.2, U2.MUTE; no longer R39.1, R84.2, R91.2, R92.2
- net N$39: now also R19.2, U2.N_OUT; no longer B_R_E1.PAD, C52.1, C56.1, R60.1, U1.BIAS_M
- net N$4: now also U1.N_OUT; no longer U8.N_OUT
- net N$41: now also C44.2, R22.1, R23.1, U2.IN+; no longer IC11B.OUT, R91.1, U$20G$1.1_2, U$20G$1.1_3
- net N$42: now also C45.2, R24.2; no longer R30.2, U$20G$1.1_1
- net N$43: now also R24.1, R26.A, U2.IN-; no longer IC10A.OUT, R19.1, R21.2
- net N$44: now also R25.2, R26.E, R26.S; no longer C10.2, R32.2, U$8.2
- net N$46: now also N_S2.PAD, PR3.1; no longer IC11A.-IN, R25.1, R26.2
- net N$5: now also C6.2, R2.2, U4.BIAS_P; no longer C9.1, IC12A.OUT, U$18G$1.1_2, U$18G$1.1_3
- net N$6: now also B_R_E1.PAD, C6.1, C8.1, R3.1, U4.BIAS_M; no longer IC1A.-IN, R7.2, R8.1
- net N$66: now also U1.COMP; no longer U8.COMP
- net N$67: now also U1.BIAS_M; no longer U8.BIAS_M
- net N$69: now also U1.BIAS_P; no longer U8.BIAS_P
- net N$7: now also C8.2, U4.COMP; no longer C4.2, IC1A.+IN, R3.1, U$2.1
- net N$70: now also U1.P_OUT; no longer U8.P_OUT
- net N$75: now also U1.OSENSE; no longer U8.OSENSE
- net N$8: now also R5.2, U4.P_OUT; no longer B_R_C1.PAD, C54.2, R58.E, R59.1
- net N$85: now also U1.MUTE; no longer U8.MUTE
- net N$9: now also P_B1.PAD, R4.2, R6.1; no longer IC2A.-IN, R12.1, R13.2
- net V+: now also C11.1, C22.+, C24.1, C3.+, C30.+, C32.1, C36.+, C38.1, C5.1, C9.+, P_D.PAD, P_D1.PAD, P_D2.PAD, U$1.S4, U4.+VCC; no longer C46.+, C50.1, C66.+, C68.1, U8.+VCC
- net V-: now also C1.-, C10.-, C12.2, C29.-, C31.2, C37.-, C39.2, C4.2, U$1.S3, U4.-VEE; no longer C44.-, C48.2, C58.-, C60.2, C65.-, C67.2, C73.-, C75.2, U8.-VEE
Other:
- note removed: "BASS LEFT CHANNEL"
- note removed: "BASS RIGHT CHANNEL"
- note removed: "Bass Amp"
- note removed: "Left"
- note removed: "Left Amp"
- note removed: "MIDS LEFT CHANNEL"
- note removed: "MIDS RIGHT CHANNEL"
- note removed: "Mute"
- note removed: "Right"
- note removed: "TREBLE LEFT CHANNEL"
- note removed: "TREBLE RIGHT CHANNEL"
- moved on the sheet: B_R_B, B_R_B1, B_R_B2, B_R_C, B_R_C1, B_R_C2, B_R_E, B_R_E1, B_R_E2, C11, C12, C13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

Commit message: Began working on PA board.
Edited parts in Parts_Library too.
Parts:
- removed B_R_B, B_R_B1, B_R_B2, B_R_C, B_R_C1, B_R_C2, B_R_E, B_R_E1, B_R_E2: SMT_PAD_3MM, Amplifier_Parts:SMT_PAD_3MM
- removed N_B, N_B1, N_B2, N_D, N_D1, N_D2, N_S, N_S1, N_S2, P_B, P_B1, P_B2, P_D, P_D1, P_D2, P_S, P_S1, P_S2: SMT_PAD_5MM, Amplifier_Parts:SMT_PAD_5MM
- removed R25, R53, R54: 1.2k, rcl:R-US_0204/2V
- removed R26, R43, R57: (no value), pot:TRIM_EU-B25U
- removed U$1: SCREW_TERMINAL_4, Amplifier_Parts:SCREW_TERMINAL_4
- removed U4: LME49830, texas:LME49830
- added B_1, B_2, B_3, C_1, C_2, C_3, E_1, E_2, E_3, N_D_1, N_D_2, N_D_3, N_G_1, N_G_2, N_G_3, N_S_1, N_S_2, N_S_3, P_D_1, P_D_2, P_D_3, P_G_1, P_G_2, P_G_3, P_S_1, P_S_2, P_S_3: (no value), Amplifier_Parts:18AWG_HOLE
- added U3: LME49830, LME49830_1:LME49830
- added VR1, VR2, VR3, VR4, VR5, VR6: (no value), Amplifier_Parts:EVM2W
- added X1: 5566-4, con-molex:5566-4
- C1, C27, C29, C3, C30: value 100uF -> 0.1uF; device rcl:CPOL-USE2.5-6 -> rcl:C-EU050-024X044
- C10, C22, C36, C37, C9: value 100uF -> 22pF; device rcl:CPOL-USE2.5-6 -> rcl:C-EU050-024X044
- C11, C13, C15, C18, C20, C21, C25, C26, C35, C40, C41, C42, C44, C45, C5, C8: device rcl:C-EU025-024X044 -> rcl:C-EU050-024X044
- C12, C17, C24, C28, C31, C32, C38, C39, C4: value 0.1uF -> 100uF; device rcl:C-EU025-024X044 -> rcl:CPOL-USE2.5-6
- C19, C33, C34, C7: value 22pF -> 0.1uF; device rcl:C-EU025-024X044 -> rcl:C-EU050-024X044
- C6: value 22pF -> 100uF; device rcl:C-EU025-024X044 -> rcl:CPOL-USE2.5-6
- R1, R13, R14: value (none) -> 1.2k; device pot:TRIM_EU-B25U -> rcl:R-US_0204/2V
- R15: value 1.2k -> 500
- R16: value 500 -> 12k
- R17: value 12k -> 1.2k
- R19, R8: value 1.2k -> 10; device rcl:R-US_0204/2V -> rcl:R-US_0309/V
- R20, R7: value 10 -> 1.2k
- R3: value 500 -> 1.2k
- R4: value 12k -> 500
- R5: value 1.2k -> 12k
- R51: device rcl:R-US_0204/2V -> rcl:R-US_0309/V
- U1, U2: device texas:LME49830 -> LME49830_1:LME49830
Connections:
- removed net MUTE1: R8.1
- removed net MUTE2: R21.1
- removed net N$10: J1.1, R54.2
- removed net N$21: R12.2, R13.E, R13.S
- removed net N$29: J1.3, R23.2
- removed net N$34: PR4.2, P_S2.PAD
- removed net N$44: R25.2, R26.E, R26.S
- removed net N$46: N_S2.PAD, PR3.1
- new net BASS: J1.2, R11.2
- new net LEFT: J1.3, R22.2
- new net N$3: C20.2, R3.2, U2.BIASP
- new net N$45: PR3.1, P_D_3.>NAME
- new net N$77: PR3.2, PR4.1, R19.2, R24.1, U$17.S4, U3.ONSENSE
- new net RIGHT: J1.1, R1.2
- net GND: now also C1.1, C12.-, C14.+, C16.+, C17.-, C18.1, C19.2, C23.-, C24.+, C25.2, C27.1, C28.-, C29.1, C3.1, C30.1, C31.+, C32.-, C33.1, C34.2, C38.-, C39.+, C4.-, C40.2, C6.-, C7.1, R10.2, R2.2, R21.2, U3.GND, X1-2.S; no longer C1.+, C10.+, C12.1, C14.-, C16.-, C17.1, C18.2, C22.-, C23.+, C24.2, C25.1, C27.-, C28.1, C29.+, C3.-, C30.-, C31.1, C32.2, C36.-, C37.+, C38.2, C39.1, C4.1, C40.1, C9.-, R22.2, R53.2, R9.2, U$1.S2, U4.GND
- net MUTE: now also R20.1, R9.1, X1-1.S; no longer U$1.S1
- net N$1: now also C21.2, C_2.>NAME, R3.1, VR4.C; no longer B_R_C1.PAD, C7.2, R1.E, R2.1
- net N$11: now also N_S_2.>NAME, PR2.2; no longer N_B1.PAD, R4.1, R5.1
- net N$110: now also P_D_1.>NAME; no longer N_S.PAD
- net N$12: now also PR1.2, PR2.1, R13.1, R8.2, U$17.S2, U2.ONSENSE; no longer PR2.2, P_S1.PAD
- net N$13: now also C27.2, R8.1; no longer PR1.2, PR2.1, R12.1, R7.2, U$17.S2, U4.OSENSE
- net N$14: now also C28.+, R9.2, U2.MUTE; no longer C13.2, R7.1
- net N$15: now also R7.2, U2.NOUT; no longer C14.+, R8.2, U4.MUTE
- net N$16: now also C1.2, R1.1, R2.1; no longer C40.2, R53.1, R54.1
- net N$17: now also C29.2, R10.1, R11.1, U2.IN+; no longer R6.2, U4.N_OUT
- net N$18: now also C30.2, R12.2; no longer C15.2, R10.1, R9.1, U4.IN+
- net N$19: now also R12.1, U2.IN-, VR3.A; no longer C28.2, R11.2
- net N$2: now also B_2.>NAME, C21.1, R4.2, VR4.A, VR4.B; no longer B_R_B1.PAD, C7.1, R1.A, R1.S, R3.2
- net N$20: now also R13.2, VR3.B, VR3.C; no longer R11.1, R13.A, U4.IN-
- net N$22: now also PR1.1, P_D_2.>NAME; no longer J1.2, R10.2
- net N$23: now also C36.2, C_3.>NAME, R14.1, VR6.C; no longer N_S1.PAD, PR1.1
- net N$24: now also B_3.>NAME, C36.1, R15.2, VR6.A, VR6.B; no longer B_R_C2.PAD, C34.2, R14.E, R15.1
- net N$25: now also C35.2, R14.2, U3.BIASP; no longer B_R_B2.PAD, C34.1, R14.A, R14.S, R16.2
- net N$26: now also C35.1, C37.1, E_3.>NAME, R15.1, U3.BIASM; no longer C33.2, R15.2, U2.BIAS_P
- net N$27: now also C37.2, U3.COMP; no longer B_R_E2.PAD, C33.1, C35.1, R16.1, U2.BIAS_M
- net N$28: now also R17.2, U3.POUT; no longer C35.2, U2.COMP
- net N$30: now also N_G_3.>NAME, R16.2, R18.1; no longer R18.2, U2.P_OUT
- net N$31: now also VR1.A; no longer R57.A
- net N$32: now also P_G_3.>NAME, R16.1, R17.1; no longer P_B2.PAD, R17.2, R19.1
- net N$33: now also N_S_3.>NAME, PR4.2; no longer N_B2.PAD, R17.1, R18.1
- net N$35: now also C42.2, R19.1; no longer PR3.2, PR4.1, R20.2, R25.1, U$17.S4, U2.OSENSE
- net N$36: now also C7.2; no longer C42.2
- net N$37: now also C43.+, R20.2, U3.MUTE; no longer C41.2, R20.1
- net N$38: now also R18.2, U3.NOUT; no longer C43.+, R21.2, U2.MUTE
- net N$39: now also C44.2, R21.1, R22.1, U3.IN+; no longer R19.2, U2.N_OUT
- net N$4: now also U1.NOUT; no longer U1.N_OUT
- net N$40: now also VR1.B, VR1.C; no longer R57.E, R57.S
- net N$41: now also C45.2, R23.2; no longer C44.2, R22.1, R23.1, U2.IN+
- net N$42: now also R23.1, U3.IN-, VR5.A; no longer C45.2, R24.2
- net N$43: now also R24.2, VR5.B, VR5.C; no longer R24.1, R26.A, U2.IN-
- net N$5: now also C20.1, C22.1, E_2.>NAME, R4.1, U2.BIASM; no longer C6.2, R2.2, U4.BIAS_P
- net N$6: now also C22.2, U2.COMP; no longer B_R_E1.PAD, C6.1, C8.1, R3.1, U4.BIAS_M
- net N$65: now also C10.2, C_1.>NAME, VR2.C; no longer B_R_C.PAD, C20.2, R43.E
- net N$66: now also C8.2; no longer C21.2
- net N$67: now also C8.1, C9.1, E_1.>NAME, U1.BIASM; no longer B_R_E.PAD, C19.1, C21.1, U1.BIAS_M
- net N$68: now also B_1.>NAME, C10.1, VR2.A, VR2.B; no longer B_R_B.PAD, C20.1, R43.A, R43.S
- net N$69: now also C9.2, U1.BIASP; no longer C19.2, U1.BIAS_P
- net N$7: now also R6.2, U2.POUT; no longer C8.2, U4.COMP
- net N$70: now also U1.POUT; no longer U1.P_OUT
- net N$72: now also N_G_1.>NAME; no longer P_B.PAD
- net N$73: now also P_G_1.>NAME; no longer N_B.PAD
- net N$74: now also N_S_1.>NAME; no longer P_S.PAD
- net N$75: now also U1.ONSENSE; no longer U1.OSENSE
- net N$8: now also N_G_2.>NAME, R7.1; no longer U4.P_OUT
- net N$84: now also C15.2; no longer C26.2
- net N$85: now also C6.+; no longer C27.+
- net N$9: now also P_G_2.>NAME, R5.1; no longer P_B1.PAD, R4.2
- net V+: now also C12.+, C17.+, C19.1, C23.+, C25.1, C32.+, C34.1, C38.+, C4.+, C40.1, N_D_1.>NAME, N_D_2.>NAME, N_D_3.>NAME, U3.+VCC, X1-4.S; no longer C16.+, C18.1, C22.+, C24.1, C3.+, C30.+, C32.1, C36.+, C38.1, C9.+, P_D.PAD, P_D1.PAD, P_D2.PAD, U$1.S4, U4.+VCC
- net V-: now also C13.2, C14.-, C16.-, C18.2, C24.-, C26.2, C3.2, C31.-, C33.2, C39.-, C41.2, P_S_1.>NAME, P_S_2.>NAME, P_S_3.>NAME, U3.-VEE, X1-3.S; no longer C1.-, C10.-, C12.2, C17.2, C23.-, C25.2, C29.-, C31.2, C37.-, C39.2, C4.2, N_D.PAD, N_D1.PAD, N_D2.PAD, U$1.S3, U4.-VEE
Other:
- moved on the sheet: C11, C13, C14, C15, C16, C18, C19, C20, C21, C23, C25, C26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
