File: Schematics/PA/Power_Amp_V1.0.sch (EAGLE design)
At the start: 99 parts, among them J1 4_PIN_AMPCONN, J11 SCREW_TERMINAL_4, J12 1725724, J13 1725724, J14 1725724, U1 LME49830, U2 LME49830, U3 LME49830

Commit message: Finished My PA and made changes to Carlos' PA
Parts:
- removed J11: SCREW_TERMINAL_4, Amplifier_Parts:SCREW_TERMINAL_4
- removed U$17: MOLEX_6P, Amplifier_Parts:MOLEX_6P
- added J2: 1984633, Amplifier_Parts:1984633
- added J3, J4, J5: 2TERMINAL_SPEAKER, Amplifier_Parts:2TERMINAL_SPEAKER
Connections:
- net BASS renamed N$1
- net GND: now also J2.1, J3.2, J4.2, J5.2; no longer J11.S1, U$17.S1, U$17.S3, U$17.S5
- net MUTE: now also J2.2; no longer J11.S2
- net N$12: now also J4.1; no longer U$17.S2
- net N$75: now also J3.1; no longer U$17.S
- net N$77: now also J5.1; no longer U$17.S4
- net V+: now also J2.4; no longer J11.S4
- net V-: now also J2.3; no longer J11.S3
Changed lines of the file:
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@@
 <setting verticaltext="up"/>
 </settings>
-<grid distance="0.1" unitdist="inch" unit="inch" style="lines" multiple="1" display="yes" altdistance="0.01" altunitdist="inch" altunit="inch"/>
+<grid distance="0.1" unitdist="inch" unit="inch" style="lines" multiple="1" display="no" altdistance="0.01" altunitdist="inch" altunit="inch"/>
 <layers>
 <layer number="1" name="Top" color="4" fill="1" visible="no" active="no"/>
@@
 <part name="GND36" library="supply2" deviceset="GND" device=""/>
 <part name="P+4" library="supply2" deviceset="V+" device=""/>
-<part name="U$17" library="Amplifier_Parts" deviceset="MOLEX_6P" device=""/>
 <part name="GND37" library="supply2" deviceset="GND" device=""/>
 <part name="FRAME1" library="frames" deviceset="FRAME_D_L" device=""/>
@@
 <part name="U2" library="LME49830_1" deviceset="LME49830" device=""/>
 <part name="U3" library="LME49830_1" deviceset="LME49830" device=""/>
-<part name="J11" library="Amplifier_Parts" deviceset="SCREW_TERMINAL_4" device=""/>
 <part name="J12" library="Amplifier_Parts" deviceset="1725724" device=""/>
 <part name="J13" library="Amplifier_Parts" deviceset="1725724" device=""/>
@@
 <part name="U$46" library="Amplifier_Parts" deviceset="SIGNAL_ARROW" device=""/>
 <part name="U$47" library="Amplifier_Parts" deviceset="SIGNAL_ARROW" device=""/>
+<part name="J2" library="Amplifier_Parts" deviceset="1984633" device=""/>
+<part name="J3" library="Amplifier_Parts" deviceset="2TERMINAL_SPEAKER" device=""/>
+<part name="J4" library="Amplifier_Parts" deviceset="2TERMINAL_SPEAKER" device=""/>
+<part name="J5" library="Amplifier_Parts" deviceset="2TERMINAL_SPEAKER" device=""/>
 </parts>
 <sheets>
@@
 </instance>
 <instance part="P+4" gate="1" x="360.68" y="426.72"/>
-<instance part="U$17" gate="G$1" x="558.8" y="238.76"/>
 <instance part="GND37" gate="GND" x="543.56" y="210.82" smashed="yes">
 <attribute name="VALUE" x="539.115" y="212.725" size="1.778" layer="96"/>
@@
 <instance part="U2" gate="G$1" x="340.36" y="208.28"/>
 <instance part="U3" gate="G$1" x="340.36" y="88.9"/>
-<instance part="J11" gate="G$1" x="40.64" y="523.24" rot="R180"/>
 <instance part="J12" gate="G$1" x="553.72" y="373.38"/>
 <instance part="J13" gate="G$1" x="624.84" y="279.4"/>
@@
 <instance part="U$46" gate="G$1" x="558.8" y="137.16"/>
 <instance part="U$47" gate="G$1" x="558.8" y="132.08"/>
+<instance part="J2" gate="G$1" x="35.56" y="518.16" rot="R180"/>
+<instance part="J3" gate="G$1" x="556.26" y="243.84"/>
+<instance part="J4" gate="G$1" x="556.26" y="233.68"/>
+<instance part="J5" gate="G$1" x="556.26" y="223.52"/>
 </instances>
 <busses>
@@
 <wire x1="497.84" y1="373.38" x2="497.84" y2="243.84" width="0.1524" layer="91"/>
 <junction x="477.52" y="373.38"/>
-<pinref part="U$17" gate="G$1" pin="S"/>
 <wire x1="497.84" y1="243.84" x2="551.18" y2="243.84" width="0.1524" layer="91"/>
 <pinref part="U1" gate="G$1" pin="ONSENSE"/>
+<pinref part="J3" gate="G$1" pin="1"/>
 </segment>
 </net>
@@
 </segment>
 <segment>
-<pinref part="U$17" gate="G$1" pin="S5"/>
 <pinref part="GND37" gate="GND" pin="GND"/>
 <wire x1="551.18" y1="218.44" x2="543.56" y2="218.44" width="0.1524" layer="91"/>
 <wire x1="543.56" y1="218.44" x2="543.56" y2="213.36" width="0.1524" layer="91"/>
-<pinref part="U$17" gate="G$1" pin="S3"/>
 <wire x1="551.18" y1="228.6" x2="543.56" y2="228.6" width="0.1524" layer="91"/>
 <wire x1="543.56" y1="228.6" x2="543.56" y2="218.44" width="0.1524" layer="91"/>
 <junction x="543.56" y="218.44"/>
-<pinref part="U$17" gate="G$1" pin="S1"/>
 <wire x1="551.18" y1="238.76" x2="543.56" y2="238.76" width="0.1524" layer="91"/>
 <wire x1="543.56" y1="238.76" x2="543.56" y2="228.6" width="0.1524" layer="91"/>
 <junction x="543.56" y="228.6"/>
+<pinref part="J3" gate="G$1" pin="2"/>
+<pinref part="J4" gate="G$1" pin="2"/>
+<pinref part="J5" gate="G$1" pin="2"/>
 </segment>
 <segment>
@@
 <pinref part="GND20" gate="GND" pin="GND"/>
 <wire x1="40.64" y1="513.08" x2="43.18" y2="513.08" width="0.1524" layer="91"/>
-<pinref part="J11" gate="G$1" pin="S1"/>
+<pinref part="J2" gate="G$1" pin="1"/>
 </segment>
 <segment>
@@
 <wire x1="60.96" y1="523.24" x2="60.96" y2="518.16" width="0.1524" layer="91"/>
 <pinref part="SUPPLY13" gate="1" pin="V-"/>
-<pinref part="J11" gate="G$1" pin="S3"/>
+<pinref part="J2" gate="G$1" pin="3"/>
 </segment>
 <segment>
@@
 <wire x1="50.8" y1="528.32" x2="50.8" y2="535.94" width="0.1524" layer="91"/>
 <pinref part="P+7" gate="1" pin="V+"/>
-<pinref part="J11" gate="G$1" pin="S4"/>
+<pinref part="J2" gate="G$1" pin="4"/>
 </segment>
 <segment>
@@
 </segment>
 <segment>
-<pinref part="J11" gate="G$1" pin="S2"/>
 <wire x1="40.64" y1="518.16" x2="48.26" y2="518.16" width="0.1524" layer="91"/>
+<pinref part="J2" gate="G$1" pin="2"/>
 </segment>
 </net>
@@
 <net name="N$77" class="0">
 <segment>
-<pinref part="U$17" gate="G$1" pin="S4"/>
 <wire x1="497.84" y1="114.3" x2="497.84" y2="223.52" width="0.1524" layer="91"/>
 <wire x1="497.84" y1="223.52" x2="551.18" y2="223.52" width="0.1524" layer="91"/>
@@
 <junction x="477.52" y="114.3"/>
 <pinref part="U3" gate="G$1" pin="ONSENSE"/>
+<pinref part="J5" gate="G$1" pin="1"/>
 </segment>
 </net>
@@
 <pinref part="PR2" gate="G$1" pin="1"/>
 <junction x="477.52" y="233.68"/>
-<pinref part="U$17" gate="G$1" pin="S2"/>
 <wire x1="477.52" y1="233.68" x2="551.18" y2="233.68" width="0.1524" layer="91"/>
 <pinref part="U2" gate="G$1" pin="ONSENSE"/>
+<pinref part="J4" gate="G$1" pin="1"/>
 </segment>
 </net>
@@
 <junction x="398.78" y="292.1"/>
 <pinref part="VR3" gate="G$1" pin="B"/>
-</segment>
-</net>
-<net name="BASS" class="0">
-<segment>
-<pinref part="R11" gate="G$1" pin="2"/>
-<wire x1="162.56" y1="233.68" x2="307.34" y2="233.68" width="0.1524" layer="91"/>
-<pinref part="J1" gate="G$1" pin="2"/>
 </segment>
 </net>
@@
 </segment>
 </net>
+<net name="N$1" class="0">
+<segment>
+<pinref part="J1" gate="G$1" pin="2"/>
+<pinref part="R11" gate="G$1" pin="2"/>
+<wire x1="162.56" y1="233.68" x2="307.34" y2="233.68" width="0.1524" layer="91"/>
+</segment>
+</net>
