File: Schematics/PA/Carlos_PA/Power_Amp_carlos.2.sch (EAGLE design)
At the start: 123 parts, among them J1 4_PIN_AMPCONN, U1 LME49830, U2 LME49830, U3 LME49830

Commit message: finished my PA board
Parts:
- removed B_1, B_2, B_3, C_1, C_2, C_3, E_1, E_2, E_3, N_D_1, N_D_2, N_D_3, N_G_1, N_G_2, N_G_3, N_S_1, N_S_2, N_S_3, P_D_1, P_D_2, P_D_3, P_G_1, P_G_2, P_G_3, P_S_1, P_S_2, P_S_3: (no value), Amplifier_Parts:18AWG_HOLE
- removed U$17: MOLEX_6P, Amplifier_Parts:MOLEX_6P
- added C46, C47, C48, C49, C50, C51, C52, C53, C54: OSTVN03A150, Amplifier_Parts:OSTVN03A150
- added U$6, U$7, U$8: 2TERMINAL_SPEAKER, Amplifier_Parts:2TERMINAL_SPEAKER
Connections:
- net GND: now also U$6.P$2, U$7.P$2, U$8.P$2; no longer U$17.S1, U$17.S3, U$17.S5
- net N$1: now also C53.1; no longer C_2.>NAME
- net N$11: now also C50.3; no longer N_S_2.>NAME
- net N$110: now also C48.1; no longer P_D_1.>NAME
- net N$12: now also U$7.P$1; no longer U$17.S2
- net N$2: now also C53.2; no longer B_2.>NAME
- net N$22: now also C49.1; no longer P_D_2.>NAME
- net N$23: now also C54.1; no longer C_3.>NAME
- net N$24: now also C54.2; no longer B_3.>NAME
- net N$26: now also C54.3; no longer E_3.>NAME
- net N$30: now also C51.2; no longer N_G_3.>NAME
- net N$32: now also C52.2; no longer P_G_3.>NAME
- net N$33: now also C51.3; no longer N_S_3.>NAME
- net N$45: now also C52.1; no longer P_D_3.>NAME
- net N$5: now also C53.3; no longer E_2.>NAME
- net N$65: now also C46.1; no longer C_1.>NAME
- net N$67: now also C46.3; no longer E_1.>NAME
- net N$68: now also C46.2; no longer B_1.>NAME
- net N$72: now also C47.2; no longer N_G_1.>NAME
- net N$73: now also C48.2; no longer P_G_1.>NAME
- net N$74: now also C47.3; no longer N_S_1.>NAME
- net N$75: now also U$6.P$1; no longer U$17.S
- net N$77: now also U$8.P$1; no longer U$17.S4
- net N$8: now also C50.2; no longer N_G_2.>NAME
- net N$9: now also C49.2; no longer P_G_2.>NAME
- net V+: now also C47.1, C50.1, C51.1; no longer N_D_1.>NAME, N_D_2.>NAME, N_D_3.>NAME
- net V-: now also C48.3, C49.3, C52.3; no longer P_S_1.>NAME, P_S_2.>NAME, P_S_3.>NAME
