File: Schematics/PA/Carlos_PA/Power_Amp_carlos.2.sch (EAGLE design)
At the start: 107 parts, among them J1 4_PIN_AMPCONN, U1 LME49830, U2 LME49830, U3 LME49830

Commit message: Finished My PA and made changes to Carlos' PA
Parts:
- removed U$5: SCREW_TERMINAL_4, Amplifier_Parts:SCREW_TERMINAL_4
- added J2: 1984633, Amplifier_Parts:1984633
- renumbered C46 to J7, C47 to J6, C48 to J8, C49 to J11, C50 to J9, C51 to J12, C52 to J14, C53 to J10, C54 to J13, U$6 to J3, U$7 to J4, U$8 to J5
Connections:
- net GND: now also J2.2, J3.2, J4.2, J5.2; no longer J3.P$2, J4.P$2, J5.P$2, U$5.S2
- net MUTE: now also J2.1; no longer U$5.S1
- net N$12: now also J4.1; no longer J4.P$1
- net N$75: now also J3.1; no longer J3.P$1
- net N$77: now also J5.1; no longer J5.P$1
- net V+: now also J2.4; no longer U$5.S4
- net V-: now also J2.3; no longer U$5.S3
