File: Schematics/PS/PowerSupply.brd (EAGLE design)
At the start: 158.8 x 110.7 mm, 79 parts, among them IC1 LM317MABDT, IC2 LM337, T1 IRFP240, T2 IRFP240

Commit message: added names to input and output traces on filter board
Parts:
- C18, C20: value 0.1uF -> 1uF
- R19: value 10k -> 120\
- R20, R21: value 10k -> 680
- R22: value 10k -> 120
Changed lines of the file:
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@@
 <element name="D11" library="Amplifier_Parts" package="1N4004" value="1N4004" x="146.0256875" y="31.1901875" rot="R270"/>
 <element name="D12" library="Amplifier_Parts" package="1N4004" value="1N4004" x="147.60016875" y="20.948165625" rot="R90"/>
-<element name="R19" library="rcl" package="0204V" value="10k" x="136.209384375" y="22.216521875" rot="R180"/>
-<element name="R20" library="rcl" package="0204V" value="10k" x="152.216559375" y="25.17390625" rot="R180"/>
+<element name="R19" library="rcl" package="0204V" value="120\" x="136.209384375" y="22.216521875" rot="R180"/>
+<element name="R20" library="rcl" package="0204V" value="680" x="152.216559375" y="25.17390625" rot="R180"/>
 <element name="C6" library="resistor" package="C025-025X050" value="10uF" x="143.111490625" y="22.441559375" rot="R180"/>
-<element name="C18" library="rcl" package="C102-064X133" value="0.1uF" x="137.92896875" y="37.884103125" rot="R270"/>
-<element name="C20" library="rcl" package="C102-064X133" value="0.1uF" x="148.706125" y="41.45679375" rot="R180"/>
+<element name="C18" library="rcl" package="C102-064X133" value="1uF" x="137.92896875" y="37.884103125" rot="R270"/>
+<element name="C20" library="rcl" package="C102-064X133" value="1uF" x="148.706125" y="41.45679375" rot="R180"/>
 <element name="D13" library="Amplifier_Parts" package="1N4004" value="1N4004" x="144.509628125" y="47.482384375" rot="R180"/>
 <element name="D14" library="Amplifier_Parts" package="1N4004" value="1N4004" x="137.829096875" y="46.109178125" rot="R90"/>
@@
 <element name="D16" library="Amplifier_Parts" package="1N4004" value="1N4004" x="144.6261" y="51.034096875" rot="R180"/>
 <element name="IC2" library="Amplifier_Parts" package="LM337" value="LM337" x="71.061990625" y="33.697915625" rot="R270"/>
-<element name="R21" library="rcl" package="0204V" value="10k" x="61.453190625" y="35.825725" rot="R180"/>
+<element name="R21" library="rcl" package="0204V" value="680" x="61.453190625" y="35.825725" rot="R180"/>
 <element name="C16" library="rcl" package="E2,5-6" value="1uF" x="150.425259375" y="28.9810875" rot="R90"/>
 <element name="C23" library="rcl" package="E2,5-6" value="1uF" x="71.78758125" y="24.378796875" rot="R90"/>
-<element name="R22" library="rcl" package="0204V" value="10k" x="60.62609375" y="31.067978125" rot="R90"/>
+<element name="R22" library="rcl" package="0204V" value="120" x="60.62609375" y="31.067978125" rot="R90"/>
 <element name="D17" library="Amplifier_Parts" package="1N4004" value="1N4004" x="63.360859375" y="33.732146875" rot="R270"/>
 <element name="C24" library="resistor" package="C025-025X050" value="10uF" x="57.080653125" y="28.268796875" rot="R90"/>

Commit message: fixed power supply board
Parts:
- added R23, R24: (no value), pot:B25P
- added R25: 390, rcl:0204V
- C1: value (none) -> 390pF
- R5: value 47k -> 23.5k
Connections:
- new net N$15: R20.1, R23.E, R23.S
- new net N$16: C13.1, D1.C, D4.C, R25.1, R7.1
- new net N$23: R21.2, R24.A
- net GND: no longer LED2.K
- net N$10: now also R25.2; no longer C13.1, D1.C, D4.C, R7.1
- net SGND: now also LED2.K, R23.A, R24.E, R24.S; no longer R20.1, R21.2
Routing:
- net N$16: track 0.00 -> 69.2 mm, vias 0 -> 1
- net N$23: track 0.00 -> 55.9 mm
- net SGND: track 84.0 -> 134.3 mm
- net N$10: track 48.6 -> 6.53 mm
- net N$15: track 0.00 -> 41.2 mm
Other:
- board size 158.8 x 110.7 mm -> 159 x 113.4 mm

Commit message: updated values on PS board
Parts:
- C14, C3: value 1uF -> 10uF
- C16, C21, C22, C23: value 1uF -> 0.1uF
- C18, C20: value 1uF -> 1nF
- R13, R14: value (none) -> 10
- R23, R24: value (none) -> 5k
- R3: value (none) -> 30k
Connections:
- net N$12 renamed SWITCH1
- net N$2 renamed SWITCH2
- net N$5 renamed NUTRAL

Commit message: added amages
Parts:
- R7: value 33 -> 330
Changed lines of the file:
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@@
 <?xml version="1.0" encoding="utf-8"?>
 <!DOCTYPE eagle SYSTEM "eagle.dtd">
-<eagle version="7.5.0">
+<eagle version="6.5.0">
 <drawing>
 <settings>
@@
 <pass name="Default">
 <param name="RoutingGrid" value="50mil"/>
-<param name="AutoGrid" value="1"/>
-<param name="Efforts" value="0"/>
-<param name="TopRouterVariant" value="1"/>
 <param name="tpViaShape" value="round"/>
 <param name="PrefDir.1" value="|"/>
@@
 <element name="R5" library="rcl" package="0617V" value="23.5k" x="73.0885" y="106.426" rot="R90"/>
 <element name="C2" library="rcl" package="C050-035X075" value="" x="83.3755" y="93.1545" rot="R90"/>
-<element name="R7" library="rcl" package="0309V" value="33" x="93.0579875" y="70.982825" rot="R180"/>
+<element name="R7" library="rcl" package="0309V" value="330" x="93.0579875" y="70.982825" rot="R180"/>
 <element name="R12" library="resistor" package="0207/15" value="100" x="153.4668" y="55.7657" rot="R90"/>
 <element name="R2" library="rcl" package="VTA52" value="2k" x="35.527175" y="56.395471875"/>
