File: Cases/carlos_case/PA.sch (EAGLE design)
At the start: 107 parts, among them J1 4_PIN_AMPCONN, J10 OSTVN03A150, J11 OSTVN03A150, J12 OSTVN03A150, J13 OSTVN03A150, J14 OSTVN03A150, J2 1984633, J3 2TERMINAL_SPEAKER, J4 2TERMINAL_SPEAKER, J5 2TERMINAL_SPEAKER, J6 OSTVN03A150, J7 OSTVN03A150, J8 OSTVN03A150, J9 OSTVN03A150, U1 LME49830, U2 LME49830, U3 LME49830

Commit message: added folder for my case
Parts:
- removed C11, C13, C25, C26, C40, C41: 0.1uF, rcl:C-EU050-024X044
- removed C12, C14, C23, C24, C38, C39: 100uF, rcl:CPOL-USE2.5-6
- removed J10, J11, J12, J13, J14, J6, J7, J8, J9: OSTVN03A150, Amplifier_Parts:OSTVN03A150
Connections:
- net BASS_IN renamed N$1
- net RIGHT_IN renamed N$2
- net B_NMOS_G: no longer J10.2
- net B_NMOS_S: no longer J10.3
- net B_PMOS_G: no longer J9.2
- net B_PMOS_S: no longer J9.1
- net B_VBE_B: no longer J11.2
- net B_VBE_C: no longer J11.3
- net B_VBE_E: no longer J11.1
- net GND: no longer C11.2, C12.-, C13.1, C14.+, C23.-, C24.+, C25.2, C26.1, C38.-, C39.+, C40.2, C41.1
- net L_NMOS_G: no longer J12.2
- net L_NMOS_S: no longer J12.3
- net L_PMOS_G: no longer J13.2
- net L_PMOS_S: no longer J13.1
- net L_VBE_B: no longer J14.2
- net L_VBE_C: no longer J14.3
- net L_VBE_E: no longer J14.1
- net R_NMOS_G: no longer J6.2
- net R_NMOS_S: no longer J6.3
- net R_PMOS_G: no longer J8.2
- net R_PMOS_S: no longer J8.1
- net R_VBE_B: no longer J7.2
- net R_VBE_C: no longer J7.3
- net R_VBE_E: no longer J7.1
- net V+: no longer C11.1, C12.+, C23.+, C25.1, C38.+, C40.1, J10.1, J12.1, J6.1
- net V-: no longer C13.2, C14.-, C24.-, C26.2, C39.-, C41.2, J13.3, J8.3, J9.3
Other:
- note removed: "250V"
- note removed: "B_PMOS_D"
- note removed: "L_NMOS_D"
- note removed: "L_PMOS_D"
- note removed: "MOSFET_n"
- note removed: "MOSFET_p"
- note removed: "R_NMOS_D"
- note removed: "R_PMOS_D"
- note removed: "Vbe multiplier"
- note removed: "altleast 2W"
- note removed: "change footprint"
