File: Cases/carlos_case/filters.brd (EAGLE design)
At the start: 101 x 47.9 mm, 112 parts, among them IC1 NE5532N, IC2 NE5532N, IC3 NE5532N, IC4 NE5532N, IC5 NE5532N, IC6 NE5532N, IC7 NE5532N, J1 3_PIN_AMPCONN, J2 4_PIN_AMPCONN, J3 3_PIN_AMPCONN

Commit message: added folder for my case
Parts:
- removed C29, C31, C33, C35, C37, C39, C41, C43, C45, C47, C49, C51, C53, C55: 0.1uF, rcl:C050-024X044
- removed C36, C38: 100uF, rcl:E2,5-6
- removed J3: 3_PIN_AMPCONN, Amplifier_Parts:3_PIN_AMPCONN
- R21, R8: value 1.2k -> 3.9k
Connections:
- net N$10 renamed RIGHT
- net N$108 renamed LEFT_IN
- net N$19 renamed BASS
- net N$26 renamed RIGHT_IN
- net N$38 renamed LEFT
- removed net +12V: C31.2, C35.2, C36.+, C39.2, C43.2, C47.2, C51.2, C55.2, IC1.8, IC2.8, IC3.8, IC4.8, IC5.8, IC6.8, IC7.8, J3.2
- removed net -12V: C29.1, C33.1, C37.1, C38.-, C41.1, C45.1, C49.1, C53.1, IC1.4, IC2.4, IC3.4, IC4.4, IC5.4, IC6.4, IC7.4, J3.1
- new net N$10: IC7.1, R19.2
- new net V+: IC1.8, IC2.8, IC3.8, IC4.8, IC5.8, IC6.8, IC7.8
- new net V-: IC1.4, IC2.4, IC3.4, IC4.4, IC5.4, IC6.4, IC7.4
- net GND: now also R47.1; no longer C29.2, C31.1, C33.2, C35.1, C36.-, C37.2, C38.+, C39.1, C41.2, C43.1, C45.2, C47.1, C49.2, C51.1, C53.2, C55.1, J3.3, VR2.P$3, VR2.P$4, VR3.P$3, VR3.P$4, VR4.P$3, VR4.P$4
- net N$43: no longer IC7.1, R19.2
- net N$63: no longer C4.1
Routing:
- net +12V: track 125.2 -> 0.00 mm
- net -12V: track 119.4 -> 0.00 mm
- net N$43: track 16.3 -> 0.00 mm
- net N$10: track 0.00 -> 14.1 mm
- net N$63: track 27.6 -> 21.9 mm
- net LEFT: track 92.4 -> 87.5 mm
- net N$5: track 18.1 -> 14.3 mm
- net N$2: track 32.9 -> 29.3 mm
- net N$22: track 7.12 -> 5.21 mm
- net N$60: track 13.9 -> 12.0 mm
- net LEFT_IN: track 4.39 -> 2.49 mm
- net N$61: track 33.0 -> 31.4 mm
- net N$40: track 36.1 -> 34.6 mm
